File: Bottom_Display.kicad_sch (KiCad schematic)
At the start: 69 parts, among them Q10 HL-2302V, Q11 HL-2302V, Q12 HL-2302V, Q13 HL-2302V, Q8 HL-2302V, Q9 HL-2302V

Commit message: Made a new hardware revision
Parts:
- removed D1, D10, D11, D12, D13, D14, D15, D16, D17, D18, D19, D2, D20, D21, D22, D23, D24, D25, D26, D27, D28, D29, D3, D30, D31, D32, D33, D34, D35, D36, D37, D38, D39, D4, D5, D6, D7, D8, D9: LED_RGAB, User_Footprints:RGB_LED_NH-B2020RGBA-HF, symbol User_Symbols:LED_RGAB
- removed Q10, Q11, Q12, Q13, Q8, Q9: HL-2302V, Package_TO_SOT_SMD:SOT-23, symbol User_Symbols:HL-2302V
- removed R12, R3, R6: 62, Resistor_SMD:R_0603_1608Metric, symbol Device:R
- removed R13, R4, R7: 36, Resistor_SMD:R_0603_1608Metric, symbol Device:R
- removed R14, R5, R8: 43, Resistor_SMD:R_0603_1608Metric, symbol Device:R
- removed R15: 21, Resistor_SMD:R_0603_1608Metric, symbol Device:R
- removed R16, R18: 20, Resistor_SMD:R_1210_3225Metric, symbol Device:R
- removed R17: 12, Resistor_SMD:R_0603_1608Metric, symbol Device:R
- removed R19: 15, Resistor_SMD:R_0603_1608Metric, symbol Device:R
- removed R20, R21: 12, Resistor_SMD:R_1210_3225Metric, symbol Device:R
- removed R22, R23: 15, Resistor_SMD:R_1210_3225Metric, symbol Device:R
- removed R40, R41, R42, R43, R44, R45: 1K, Resistor_SMD:R_0603_1608Metric, symbol Device:R
- added D10, D11, D12, D14, D15, D153, D154, D155, D156, D16, D17, D18, D19, D2, D22, D23, D24, D25, D27, D28, D29, D3, D30, D31, D32, D33, D34, D35, D36, D37, D38, D39, D4, D40, D5, D6, D7, D8, D9: (no value), symbol LED:WS2812B
Connections:
- new net: D27.4 (DIN), D38.2 (DOUT)
- new net: D37.2 (DOUT), D38.4 (DIN)
- new net: D28.4 (DIN), D40.2 (DOUT)
- new net: D39.2 (DOUT), D40.4 (DIN)
- new net: D36.2 (DOUT), D37.4 (DIN)
- new net: D156.2 (DOUT), D36.4 (DIN)
- new net: D17.4 (DIN), D2.2 (DOUT)
- new net: D2.4 (DIN), D3.2 (DOUT)
- new net: D29.2 (DOUT), D39.4 (DIN)
- new net: D153.2 (DOUT), D3.4 (DIN)
- new net: D19.4 (DIN), D24.2 (DOUT)
- new net: D24.4 (DIN), D28.2 (DOUT)
- new net: D10.4 (DIN), D14.2 (DOUT)
- new net: D14.4 (DIN), D18.2 (DOUT)
- new net: D154.4 (DIN), D8.2 (DOUT)
- new net: D8.4 (DIN), D9.2 (DOUT)
- new net: D6.4 (DIN), D7.2 (DOUT)
- new net: D154.2 (DOUT), D7.4 (DIN)
- new net: D22.2 (DOUT), D25.4 (DIN)
- new net: D16.2 (DOUT), D22.4 (DIN)
- new net: D156.4 (DIN), D35.2 (DOUT)
- new net: D34.2 (DOUT), D35.4 (DIN)
- new net: D4.4 (DIN), D5.2 (DOUT)
- new net: D5.4 (DIN), D6.2 (DOUT)
- new net: D155.2 (DOUT), D32.4 (DIN)
- new net: D155.4 (DIN), D31.2 (DOUT)
- new net: D32.2 (DOUT), D33.4 (DIN)
- new net: D10.2 (DOUT), D11.4 (DIN)
- new net: D33.2 (DOUT), D34.4 (DIN)
- new net: D18.4 (DIN), D23.2 (DOUT)
- new net: D11.2 (DOUT), D16.4 (DIN)
- new net: D12.4 (DIN), D15.2 (DOUT)
- new net: D17.2 (DOUT), D30.4 (DIN)
- new net: D15.4 (DIN), D19.2 (DOUT)
- new net: D30.2 (DOUT), D31.4 (DIN)
- new net: D23.4 (DIN), D27.2 (DOUT)
- new net: D25.2 (DOUT), D29.4 (DIN)
- new net: D153.4 (DIN), D4.2 (DOUT)
- new net E1_DIN: D9.4 (DIN)
- new net E_VDD: D10.1 (VDD), D11.1 (VDD), D12.1 (VDD), D14.1 (VDD), D15.1 (VDD), D153.1 (VDD), D154.1 (VDD), D155.1 (VDD), D156.1 (VDD), D16.1 (VDD), D17.1 (VDD), D18.1 (VDD), D19.1 (VDD), D2.1 (VDD), D22.1 (VDD), D23.1 (VDD), D24.1 (VDD), D25.1 (VDD), D27.1 (VDD), D28.1 (VDD), D29.1 (VDD), D3.1 (VDD), D30.1 (VDD), D31.1 (VDD), D32.1 (VDD), D33.1 (VDD), D34.1 (VDD), D35.1 (VDD), D36.1 (VDD), D37.1 (VDD), D38.1 (VDD), D39.1 (VDD), D4.1 (VDD), D40.1 (VDD), D5.1 (VDD), D6.1 (VDD), D7.1 (VDD), D8.1 (VDD), D9.1 (VDD)
- new net E_VSS: D10.3 (VSS), D11.3 (VSS), D12.3 (VSS), D14.3 (VSS), D15.3 (VSS), D153.3 (VSS), D154.3 (VSS), D155.3 (VSS), D156.3 (VSS), D16.3 (VSS), D17.3 (VSS), D18.3 (VSS), D19.3 (VSS), D2.3 (VSS), D22.3 (VSS), D23.3 (VSS), D24.3 (VSS), D25.3 (VSS), D27.3 (VSS), D28.3 (VSS), D29.3 (VSS), D3.3 (VSS), D30.3 (VSS), D31.3 (VSS), D32.3 (VSS), D33.3 (VSS), D34.3 (VSS), D35.3 (VSS), D36.3 (VSS), D37.3 (VSS), D38.3 (VSS), D39.3 (VSS), D4.3 (VSS), D40.3 (VSS), D5.3 (VSS), D6.3 (VSS), D7.3 (VSS), D8.3 (VSS), D9.3 (VSS)
- no-connect marks 36 -> 0

Commit message: new version with indexed leds
Parts:
- D10, D11, D12, D14, D15, D153, D154, D155, D156, D16, D17, D18, D19, D2, D22, D23, D24, D25, D27, D28, D29, D3, D30, D31, D32, D33, D34, D35, D36, D37, D38, D39, D4, D40, D5, D6, D7, D8, D9: value (none) -> LED_WS2812B; footprint (none) -> User_Footprints:LED_WS2812B_2x1.8mm; Manufacturer (none) -> TUOZHAN; Notes (none) -> 5mA; Package SMD-4P, 5x5mm -> led 3227; Part Number XL-5050RGBC-WS2812B-S -> TZ-0807Z1RGB-5V-I4-MS(5mA); Price .0228 -> .0288; Website https://www.lcsc.com/product-detail/RGB-LEDs-Built-in-IC_XI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 -> https://www.lcsc.com/product-detail/RGB-LEDs-Built-in-IC_TU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
