File: Left_Display.kicad_sch (KiCad schematic)
At the start: 74 parts, among them Q20 HL-2302V, Q21 HL-2302V, Q22 HL-2302V, Q23 HL-2302V, Q24 HL-2302V, Q25 HL-2302V

Commit message: Made a new hardware revision
Parts:
- removed D113, D114, D115, D116, D117, D118, D119, D120, D121, D122, D123, D124, D125, D126, D127, D128, D129, D130, D131, D132, D133, D134, D135, D136, D137, D138, D139, D140, D141, D142, D143, D144, D145, D146, D147, D148, D149, D150, D151, D152, D153, D154, D155, D156, D157, D158, D159, D160, D161, D162, D163, D164, D165, D166, D167, D168: LED_RGAB, User_Footprints:RGB_LED_NH-B2020RGBA-HF, symbol User_Symbols:LED_RGAB
- removed Q20, Q21, Q22, Q23, Q24, Q25: HL-2302V, Package_TO_SOT_SMD:SOT-23, symbol User_Symbols:HL-2302V
- removed R10, R31: 12, Resistor_SMD:R_1210_3225Metric, symbol Device:R
- removed R11, R32: 15, Resistor_SMD:R_1210_3225Metric, symbol Device:R
- removed R30, R9: 20, Resistor_SMD:R_1210_3225Metric, symbol Device:R
- removed R52, R53, R54, R55, R56, R57: 1K, Resistor_SMD:R_0603_1608Metric, symbol Device:R
- added D100, D101, D102, D103, D104, D105, D106, D107, D108, D109, D110, D111, D112, D113, D114, D115, D116, D117, D118, D119, D120, D121, D122, D123, D124, D125, D126, D127, D128, D129, D130, D131, D132, D133, D134, D135, D136, D137, D138, D139, D140, D141, D142, D143, D144, D145, D146, D147, D148, D149, D150, D151, D152, D171, D172, D173, D174, D175, D176, D177, D178, D179, D180, D181, D182, D183, D184, D20, D21, D26, D97, D98, D99: (no value), symbol LED:WS2812B
Connections:
- new net: D105.2 (DOUT), D108.4 (DIN)
- new net: D105.4 (DIN), D97.2 (DOUT)
- new net: D147.2 (DOUT), D148.4 (DIN)
- new net: D147.4 (DIN), D183.2 (DOUT)
- new net: D139.4 (DIN), D180.2 (DOUT)
- new net: D136.2 (DOUT), D180.4 (DIN)
- new net: D138.4 (DIN), D182.2 (DOUT)
- new net: D141.2 (DOUT), D182.4 (DIN)
- new net: D131.4 (DIN), D132.2 (DOUT)
- new net: D132.4 (DIN), D135.2 (DOUT)
- new net: D133.2 (DOUT), D136.4 (DIN)
- new net: D125.2 (DOUT), D133.4 (DIN)
- new net: D111.2 (DOUT), D114.4 (DIN)
- new net: D111.4 (DIN), D173.2 (DOUT)
- new net: D146.2 (DOUT), D183.4 (DIN)
- new net: D121.2 (DOUT), D122.4 (DIN)
- new net: D116.4 (DIN), D124.2 (DOUT)
- new net: D123.2 (DOUT), D124.4 (DIN)
- new net: D140.2 (DOUT), D143.4 (DIN)
- new net: D140.4 (DIN), D181.2 (DOUT)
- new net: D113.4 (DIN), D116.2 (DOUT)
- new net: D125.4 (DIN), D126.2 (DOUT)
- new net: D150.2 (DOUT), D184.4 (DIN)
- new net: D149.2 (DOUT), D150.4 (DIN)
- new net: D141.4 (DIN), D144.2 (DOUT)
- new net: D144.4 (DIN), D152.2 (DOUT)
- new net: D151.2 (DOUT), D152.4 (DIN)
- new net: D149.4 (DIN), D26.2 (DOUT)
- new net: D118.2 (DOUT), D176.4 (DIN)
- new net: D117.2 (DOUT), D118.4 (DIN)
- new net: D142.2 (DOUT), D145.4 (DIN)
- new net: D139.2 (DOUT), D142.4 (DIN)
- new net: D103.4 (DIN), D104.2 (DOUT)
- new net: D104.4 (DIN), D107.2 (DOUT)
- new net: D101.4 (DIN), D102.2 (DOUT)
- new net: D102.4 (DIN), D172.2 (DOUT)
- new net: D145.2 (DOUT), D146.4 (DIN)
- new net: D171.4 (DIN), D99.2 (DOUT)
- new net: D100.2 (DOUT), D99.4 (DIN)
- new net: D21.2 (DOUT), D26.4 (DIN)
- new net: D148.2 (DOUT), D21.4 (DIN)
- new net: D123.4 (DIN), D177.2 (DOUT)
- new net: D117.4 (DIN), D20.2 (DOUT)
- new net: D135.4 (DIN), D138.2 (DOUT)
- new net: D127.4 (DIN), D128.2 (DOUT)
- new net: D114.2 (DOUT), D20.4 (DIN)
- new net: D107.4 (DIN), D110.2 (DOUT)
- new net: D110.4 (DIN), D175.2 (DOUT)
- new net: D113.2 (DOUT), D175.4 (DIN)
- new net: D122.2 (DOUT), D177.4 (DIN)
- new net: D103.2 (DOUT), D172.4 (DIN)
- new net: D97.4 (DIN), D98.2 (DOUT)
- new net: D171.2 (DOUT), D98.4 (DIN)
- new net: D137.2 (DOUT), D181.4 (DIN)
- new net: D134.2 (DOUT), D137.4 (DIN)
- new net: D100.4 (DIN), D101.2 (DOUT)
- new net: D131.2 (DOUT), D179.4 (DIN)
- new net: D108.2 (DOUT), D173.4 (DIN)
- new net: D119.2 (DOUT), D120.4 (DIN)
- new net: D119.4 (DIN), D176.2 (DOUT)
- new net: D129.2 (DOUT), D134.4 (DIN)
- new net: D129.4 (DIN), D130.2 (DOUT)
- new net: D109.2 (DOUT), D174.4 (DIN)
- new net: D106.2 (DOUT), D109.4 (DIN)
- new net: D112.2 (DOUT), D115.4 (DIN)
- new net: D112.4 (DIN), D174.2 (DOUT)
- new net: D127.2 (DOUT), D178.4 (DIN)
- new net: D106.4 (DIN), D120.2 (DOUT)
- new net: D126.4 (DIN), D178.2 (DOUT)
- new net: D151.4 (DIN), D184.2 (DOUT)
- new net: D130.4 (DIN), D179.2 (DOUT)
- new net L1_DIN: D121.4 (DIN)
- new net L2_DIN: D128.4 (DIN)
- new net L_VDD: D100.1 (VDD), D101.1 (VDD), D102.1 (VDD), D103.1 (VDD), D104.1 (VDD), D105.1 (VDD), D106.1 (VDD), D107.1 (VDD), D108.1 (VDD), D109.1 (VDD), D110.1 (VDD), D111.1 (VDD), D112.1 (VDD), D113.1 (VDD), D114.1 (VDD), D115.1 (VDD), D116.1 (VDD), D117.1 (VDD), D118.1 (VDD), D119.1 (VDD), D120.1 (VDD), D121.1 (VDD), D122.1 (VDD), D123.1 (VDD), D124.1 (VDD), D125.1 (VDD), D126.1 (VDD), D127.1 (VDD), D128.1 (VDD), D129.1 (VDD), D130.1 (VDD), D131.1 (VDD), D132.1 (VDD), D133.1 (VDD), D134.1 (VDD), D135.1 (VDD), D136.1 (VDD), D137.1 (VDD), D138.1 (VDD), D139.1 (VDD), D140.1 (VDD), D141.1 (VDD), D142.1 (VDD), D143.1 (VDD), D144.1 (VDD), D145.1 (VDD), D146.1 (VDD), D147.1 (VDD), D148.1 (VDD), D149.1 (VDD), D150.1 (VDD), D151.1 (VDD), D152.1 (VDD), D171.1 (VDD), D172.1 (VDD), D173.1 (VDD), D174.1 (VDD), D175.1 (VDD), D176.1 (VDD), D177.1 (VDD), D178.1 (VDD), D179.1 (VDD), D180.1 (VDD), D181.1 (VDD), D182.1 (VDD), D183.1 (VDD), D184.1 (VDD), D20.1 (VDD), D21.1 (VDD), D26.1 (VDD), D97.1 (VDD), D98.1 (VDD), D99.1 (VDD)
- new net L_VSS: D100.3 (VSS), D101.3 (VSS), D102.3 (VSS), D103.3 (VSS), D104.3 (VSS), D105.3 (VSS), D106.3 (VSS), D107.3 (VSS), D108.3 (VSS), D109.3 (VSS), D110.3 (VSS), D111.3 (VSS), D112.3 (VSS), D113.3 (VSS), D114.3 (VSS), D115.3 (VSS), D116.3 (VSS), D117.3 (VSS), D118.3 (VSS), D119.3 (VSS), D120.3 (VSS), D121.3 (VSS), D122.3 (VSS), D123.3 (VSS), D124.3 (VSS), D125.3 (VSS), D126.3 (VSS), D127.3 (VSS), D128.3 (VSS), D129.3 (VSS), D130.3 (VSS), D131.3 (VSS), D132.3 (VSS), D133.3 (VSS), D134.3 (VSS), D135.3 (VSS), D136.3 (VSS), D137.3 (VSS), D138.3 (VSS), D139.3 (VSS), D140.3 (VSS), D141.3 (VSS), D142.3 (VSS), D143.3 (VSS), D144.3 (VSS), D145.3 (VSS), D146.3 (VSS), D147.3 (VSS), D148.3 (VSS), D149.3 (VSS), D150.3 (VSS), D151.3 (VSS), D152.3 (VSS), D171.3 (VSS), D172.3 (VSS), D173.3 (VSS), D174.3 (VSS), D175.3 (VSS), D176.3 (VSS), D177.3 (VSS), D178.3 (VSS), D179.3 (VSS), D180.3 (VSS), D181.3 (VSS), D182.3 (VSS), D183.3 (VSS), D184.3 (VSS), D20.3 (VSS), D21.3 (VSS), D26.3 (VSS), D97.3 (VSS), D98.3 (VSS), D99.3 (VSS)

Commit message: new version with indexed leds
Parts:
- D100, D101, D102, D103, D104, D105, D106, D107, D108, D109, D110, D111, D112, D113, D114, D115, D116, D117, D118, D119, D120, D121, D122, D123, D124, D125, D126, D127, D128, D129, D130, D131, D132, D133, D134, D135, D136, D137, D138, D139, D140, D141, D142, D143, D144, D145, D146, D147, D148, D149, D150, D151, D152, D171, D172, D173, D174, D175, D176, D177, D178, D179, D180, D181, D182, D183, D184, D20, D21, D26, D97, D98, D99: value (none) -> LED_WS2812B; footprint (none) -> User_Footprints:LED_WS2812B_2x1.8mm; Manufacturer (none) -> TUOZHAN; Notes (none) -> 5mA; Package SMD-4P, 5x5mm -> led 3227; Part Number XL-5050RGBC-WS2812B-S -> TZ-0807Z1RGB-5V-I4-MS(5mA); Price .0228 -> .0288; Website https://www.lcsc.com/product-detail/RGB-LEDs-Built-in-IC_XI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 -> https://www.lcsc.com/product-detail/RGB-LEDs-Built-in-IC_TU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
