File: Right_Display.kicad_sch (KiCad schematic)
At the start: 74 parts, among them Q14 HL-2302V, Q15 HL-2302V, Q16 HL-2302V, Q17 HL-2302V, Q18 HL-2302V, Q19 HL-2302V

Commit message: Made a new hardware revision
Parts:
- removed D100, D101, D102, D103, D104, D105, D106, D107, D108, D109, D110, D111, D112, D57, D58, D59, D60, D61, D62, D63, D64, D65, D66, D67, D68, D69, D70, D71, D72, D73, D74, D75, D76, D77, D78, D79, D80, D81, D82, D83, D84, D85, D86, D87, D88, D89, D90, D91, D92, D93, D94, D95, D96, D97, D98, D99: LED_RGAB, User_Footprints:RGB_LED_NH-B2020RGBA-HF, symbol User_Symbols:LED_RGAB
- removed Q14, Q15, Q16, Q17, Q18, Q19: HL-2302V, Package_TO_SOT_SMD:SOT-23, symbol User_Symbols:HL-2302V
- removed R24, R27: 20, Resistor_SMD:R_1210_3225Metric, symbol Device:R
- removed R25, R28: 12, Resistor_SMD:R_1210_3225Metric, symbol Device:R
- removed R26, R29: 15, Resistor_SMD:R_1210_3225Metric, symbol Device:R
- removed R46, R47, R48, R49, R50, R51: 1K, Resistor_SMD:R_0603_1608Metric, symbol Device:R
- added D13, D157, D158, D159, D160, D161, D162, D163, D164, D165, D166, D167, D168, D169, D170, D41, D42, D43, D44, D45, D46, D47, D48, D49, D50, D51, D52, D53, D54, D55, D56, D57, D58, D59, D60, D61, D62, D63, D64, D65, D66, D67, D68, D69, D70, D71, D72, D73, D74, D75, D76, D77, D78, D79, D80, D81, D82, D83, D84, D85, D86, D87, D88, D89, D90, D91, D92, D93, D94, D95, D96: (no value), symbol LED:WS2812B
Connections:
- new net: D49.2 (DOUT), D52.4 (DIN)
- new net: D41.2 (DOUT), D49.4 (DIN)
- new net: D83.2 (DOUT), D86.4 (DIN)
- new net: D166.2 (DOUT), D83.4 (DIN)
- new net: D158.2 (DOUT), D46.4 (DIN)
- new net: D158.4 (DIN), D47.2 (DOUT)
- new net: D48.4 (DIN), D51.2 (DOUT)
- new net: D51.4 (DIN), D54.2 (DOUT)
- new net: D163.2 (DOUT), D67.4 (DIN)
- new net: D163.4 (DIN), D66.2 (DOUT)
- new net: D157.4 (DIN), D43.2 (DOUT)
- new net: D43.4 (DIN), D44.2 (DOUT)
- new net: D166.4 (DIN), D80.2 (DOUT)
- new net: D41.4 (DIN), D42.2 (DOUT)
- new net: D13.2 (DOUT), D61.4 (DIN)
- new net: D13.4 (DIN), D58.2 (DOUT)
- new net: D55.2 (DOUT), D58.4 (DIN)
- new net: D160.2 (DOUT), D56.4 (DIN)
- new net: D160.4 (DIN), D53.2 (DOUT)
- new net: D47.4 (DIN), D48.2 (DOUT)
- new net: D170.4 (DIN), D94.2 (DOUT)
- new net: D93.2 (DOUT), D94.4 (DIN)
- new net: D65.2 (DOUT), D66.4 (DIN)
- new net: D164.2 (DOUT), D70.4 (DIN)
- new net: D164.4 (DIN), D71.2 (DOUT)
- new net: D157.2 (DOUT), D42.4 (DIN)
- new net: D56.2 (DOUT), D59.4 (DIN)
- new net: D169.2 (DOUT), D91.4 (DIN)
- new net: D169.4 (DIN), D90.2 (DOUT)
- new net: D159.2 (DOUT), D55.4 (DIN)
- new net: D159.4 (DIN), D52.2 (DOUT)
- new net: D73.4 (DIN), D74.2 (DOUT)
- new net: D165.2 (DOUT), D74.4 (DIN)
- new net: D77.2 (DOUT), D80.4 (DIN)
- new net: D89.2 (DOUT), D90.4 (DIN)
- new net: D86.2 (DOUT), D89.4 (DIN)
- new net: D44.4 (DIN), D45.2 (DOUT)
- new net: D63.2 (DOUT), D64.4 (DIN)
- new net: D162.2 (DOUT), D63.4 (DIN)
- new net: D78.2 (DOUT), D81.4 (DIN)
- new net: D73.2 (DOUT), D78.4 (DIN)
- new net: D84.2 (DOUT), D87.4 (DIN)
- new net: D60.4 (DIN), D68.2 (DOUT)
- new net: D67.2 (DOUT), D68.4 (DIN)
- new net: D57.4 (DIN), D60.2 (DOUT)
- new net: D92.2 (DOUT), D93.4 (DIN)
- new net: D91.2 (DOUT), D92.4 (DIN)
- new net: D161.2 (DOUT), D54.4 (DIN)
- new net: D161.4 (DIN), D57.2 (DOUT)
- new net: D167.2 (DOUT), D84.4 (DIN)
- new net: D167.4 (DIN), D81.2 (DOUT)
- new net: D71.4 (DIN), D72.2 (DOUT)
- new net: D50.4 (DIN), D64.2 (DOUT)
- new net: D170.2 (DOUT), D95.4 (DIN)
- new net: D61.2 (DOUT), D62.4 (DIN)
- new net: D162.4 (DIN), D62.2 (DOUT)
- new net: D69.2 (DOUT), D77.4 (DIN)
- new net: D50.2 (DOUT), D53.4 (DIN)
- new net: D168.4 (DIN), D85.2 (DOUT)
- new net: D85.4 (DIN), D88.2 (DOUT)
- new net: D69.4 (DIN), D70.2 (DOUT)
- new net: D165.4 (DIN), D75.2 (DOUT)
- new net: D79.4 (DIN), D82.2 (DOUT)
- new net: D168.2 (DOUT), D82.4 (DIN)
- new net: D45.4 (DIN), D46.2 (DOUT)
- new net: D76.4 (DIN), D79.2 (DOUT)
- new net: D88.4 (DIN), D96.2 (DOUT)
- new net: D95.2 (DOUT), D96.4 (DIN)
- new net: D75.4 (DIN), D76.2 (DOUT)
- new net R1_DIN: D65.4 (DIN)
- new net R2_DIN: D72.4 (DIN)
- new net R_VDD: D13.1 (VDD), D157.1 (VDD), D158.1 (VDD), D159.1 (VDD), D160.1 (VDD), D161.1 (VDD), D162.1 (VDD), D163.1 (VDD), D164.1 (VDD), D165.1 (VDD), D166.1 (VDD), D167.1 (VDD), D168.1 (VDD), D169.1 (VDD), D170.1 (VDD), D41.1 (VDD), D42.1 (VDD), D43.1 (VDD), D44.1 (VDD), D45.1 (VDD), D46.1 (VDD), D47.1 (VDD), D48.1 (VDD), D49.1 (VDD), D50.1 (VDD), D51.1 (VDD), D52.1 (VDD), D53.1 (VDD), D54.1 (VDD), D55.1 (VDD), D56.1 (VDD), D57.1 (VDD), D58.1 (VDD), D59.1 (VDD), D60.1 (VDD), D61.1 (VDD), D62.1 (VDD), D63.1 (VDD), D64.1 (VDD), D65.1 (VDD), D66.1 (VDD), D67.1 (VDD), D68.1 (VDD), D69.1 (VDD), D70.1 (VDD), D71.1 (VDD), D72.1 (VDD), D73.1 (VDD), D74.1 (VDD), D75.1 (VDD), D76.1 (VDD), D77.1 (VDD), D78.1 (VDD), D79.1 (VDD), D80.1 (VDD), D81.1 (VDD), D82.1 (VDD), D83.1 (VDD), D84.1 (VDD), D85.1 (VDD), D86.1 (VDD), D87.1 (VDD), D88.1 (VDD), D89.1 (VDD), D90.1 (VDD), D91.1 (VDD), D92.1 (VDD), D93.1 (VDD), D94.1 (VDD), D95.1 (VDD), D96.1 (VDD)
- new net R_VSS: D13.3 (VSS), D157.3 (VSS), D158.3 (VSS), D159.3 (VSS), D160.3 (VSS), D161.3 (VSS), D162.3 (VSS), D163.3 (VSS), D164.3 (VSS), D165.3 (VSS), D166.3 (VSS), D167.3 (VSS), D168.3 (VSS), D169.3 (VSS), D170.3 (VSS), D41.3 (VSS), D42.3 (VSS), D43.3 (VSS), D44.3 (VSS), D45.3 (VSS), D46.3 (VSS), D47.3 (VSS), D48.3 (VSS), D49.3 (VSS), D50.3 (VSS), D51.3 (VSS), D52.3 (VSS), D53.3 (VSS), D54.3 (VSS), D55.3 (VSS), D56.3 (VSS), D57.3 (VSS), D58.3 (VSS), D59.3 (VSS), D60.3 (VSS), D61.3 (VSS), D62.3 (VSS), D63.3 (VSS), D64.3 (VSS), D65.3 (VSS), D66.3 (VSS), D67.3 (VSS), D68.3 (VSS), D69.3 (VSS), D70.3 (VSS), D71.3 (VSS), D72.3 (VSS), D73.3 (VSS), D74.3 (VSS), D75.3 (VSS), D76.3 (VSS), D77.3 (VSS), D78.3 (VSS), D79.3 (VSS), D80.3 (VSS), D81.3 (VSS), D82.3 (VSS), D83.3 (VSS), D84.3 (VSS), D85.3 (VSS), D86.3 (VSS), D87.3 (VSS), D88.3 (VSS), D89.3 (VSS), D90.3 (VSS), D91.3 (VSS), D92.3 (VSS), D93.3 (VSS), D94.3 (VSS), D95.3 (VSS), D96.3 (VSS)

Commit message: new version with indexed leds
Parts:
- D13, D157, D158, D159, D160, D161, D162, D163, D164, D165, D166, D167, D168, D169, D170, D41, D42, D43, D44, D45, D46, D47, D48, D49, D50, D51, D52, D53, D54, D55, D56, D57, D58, D59, D60, D61, D62, D63, D64, D65, D66, D67, D68, D69, D70, D71, D72, D73, D74, D75, D76, D77, D78, D79, D80, D81, D82, D83, D84, D85, D86, D87, D88, D89, D90, D91, D92, D93, D94, D95, D96: value (none) -> LED_WS2812B; footprint (none) -> User_Footprints:LED_WS2812B_2x1.8mm; Manufacturer (none) -> TUOZHAN; Notes (none) -> 5mA; Package SMD-4P, 5x5mm -> led 3227; Part Number XL-5050RGBC-WS2812B-S -> TZ-0807Z1RGB-5V-I4-MS(5mA); Price .0228 -> .0288; Website https://www.lcsc.com/product-detail/RGB-LEDs-Built-in-IC_XI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 -> https://www.lcsc.com/product-detail/RGB-LEDs-Built-in-IC_TU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
