File: Scoreboard.kicad_pcb (KiCad board)
At the start: 2 copper layers, 140.5 x 64.5 mm, 256 parts, among them J1 TC2050-IDC-NL, P1 USB_C_Plug_USB2.0, Q1 HL-2301V, Q10 HL-2302V, Q11 HL-2302V, Q12 HL-2302V, Q13 HL-2302V, Q14 HL-2302V, Q15 HL-2302V, Q16 HL-2302V, Q17 HL-2302V, Q18 HL-2302V, Q19 HL-2302V, Q2 HL-2301V, Q20 HL-2302V, Q21 HL-2302V, Q22 HL-2302V, Q23 HL-2302V, Q24 HL-2302V, Q25 HL-2302V, Q3 HL-2301V, Q4 HL-2301V, Q5 HL-2301V, Q6 HL-2301V, Q7 HL-2301V, Q8 HL-2302V, Q9 HL-2302V, SW2 SW_Push, SW3 SW_Push, SW4 SW_Push, U1 AP63203WU, U2 BM832, U3 LM66100DCKR, U4 LM66100DCKR

Commit message: Made a new hardware revision
Parts:
- removed BT3: AA_BATTERY, User_Footprints:BAT_BCAAPC
- removed the C2 at (191.0, 78.2)
- removed C7: 1u, Capacitor_SMD:C_0603_1608Metric
- removed C8: 4u7, Capacitor_SMD:C_0603_1608Metric
- removed the D12 at (126.2, 86.6)
- removed the D30 at (145.4, 46.1)
- removed the D6 at (70.3, 46.1)
- removed L1: 4u7, Inductor_SMD:L_0603_1608Metric
- removed P1: USB_C_Plug_USB2.0, User_Footprints:DEALON_USB-TYPE-C-009
- removed Q10, Q11, Q12, Q13, Q14, Q15, Q16, Q17, Q18, Q19, Q20, Q21, Q22, Q23, Q24, Q25, Q8, Q9: HL-2302V, Package_TO_SOT_SMD:SOT-23
- removed Q5, Q6, Q7: HL-2301V, Package_TO_SOT_SMD:SOT-23
- removed R20, R21, R25, R28, R31: 12, Resistor_SMD:R_1210_3225Metric
- removed R22, R23, R26, R29, R32: 15, Resistor_SMD:R_1210_3225Metric
- removed R24, R27, R30: 20, Resistor_SMD:R_1210_3225Metric
- removed R33, R34, R35, R36, R37, R38, R39, R40, R41, R42, R43, R44, R45, R46, R47, R48, R49, R50, R51, R52, R53, R54, R55, R56, R57: 1K, Resistor_SMD:R_0603_1608Metric
- removed SW4: SW_Push, User_Footprints:SW_SPST_TSC015A03526A
- removed U2: BM832, User_Footprints:BM832
- removed U3, U4: LM66100DCKR, User_Footprints:DCK6_TEX-L
- added D169: LED_WS2812B, User_Footprints:LED_WS2812B_2x1.8mm, F.Cu at (221.4, 111.9)
- added D170: LED_WS2812B, User_Footprints:LED_WS2812B_2x1.8mm, F.Cu at (221.4, 131.8)
- added D171: LED_WS2812B, User_Footprints:LED_WS2812B_2x1.8mm, F.Cu at (97.5, 111.9)
- added D172: LED_WS2812B, User_Footprints:LED_WS2812B_2x1.8mm, F.Cu at (97.5, 131.8)
- added D173: LED_WS2812B, User_Footprints:LED_WS2812B_2x1.8mm, F.Cu at (107.5, 102.0)
- added D174: LED_WS2812B, User_Footprints:LED_WS2812B_2x1.8mm, F.Cu at (107.5, 121.8)
- added D175: LED_WS2812B, User_Footprints:LED_WS2812B_2x1.8mm, F.Cu at (107.5, 141.7)
- added D176: LED_WS2812B, User_Footprints:LED_WS2812B_2x1.8mm, F.Cu at (117.4, 111.9)
- added D177: LED_WS2812B, User_Footprints:LED_WS2812B_2x1.8mm, F.Cu at (117.5, 131.8)
- added D178: LED_WS2812B, User_Footprints:LED_WS2812B_2x1.8mm, F.Cu at (126.4, 111.9)
- added D179: LED_WS2812B, User_Footprints:LED_WS2812B_2x1.8mm, F.Cu at (126.4, 131.8)
- added D180: LED_WS2812B, User_Footprints:LED_WS2812B_2x1.8mm, F.Cu at (136.3, 102.0)
- added D181: LED_WS2812B, User_Footprints:LED_WS2812B_2x1.8mm, F.Cu at (136.3, 121.8)
- added D182: LED_WS2812B, User_Footprints:LED_WS2812B_2x1.8mm, F.Cu at (136.3, 141.7)
- added D183: LED_WS2812B, User_Footprints:LED_WS2812B_2x1.8mm, F.Cu at (146.3, 111.9)
- added D184: LED_WS2812B, User_Footprints:LED_WS2812B_2x1.8mm, F.Cu at (146.2, 131.8)
- added D37: LED_WS2812B, User_Footprints:LED_WS2812B_2x1.8mm, F.Cu at (163.8, 138.4)
- added D40: LED_WS2812B, User_Footprints:LED_WS2812B_2x1.8mm, F.Cu at (184.5, 159.4)
- added D41: LED_WS2812B, User_Footprints:LED_WS2812B_2x1.8mm, F.Cu at (172.7, 105.3)
- added D42: LED_WS2812B, User_Footprints:LED_WS2812B_2x1.8mm, F.Cu at (172.7, 108.6)
- added D43: LED_WS2812B, User_Footprints:LED_WS2812B_2x1.8mm, F.Cu at (172.7, 115.2)
- added D44: LED_WS2812B, User_Footprints:LED_WS2812B_2x1.8mm, F.Cu at (172.7, 118.5)
- added D45: LED_WS2812B, User_Footprints:LED_WS2812B_2x1.8mm, F.Cu at (172.7, 125.2)
- added D46: LED_WS2812B, User_Footprints:LED_WS2812B_2x1.8mm, F.Cu at (172.7, 128.5)
- added D47: LED_WS2812B, User_Footprints:LED_WS2812B_2x1.8mm, F.Cu at (172.7, 135.1)
- added D48: LED_WS2812B, User_Footprints:LED_WS2812B_2x1.8mm, F.Cu at (172.7, 138.4)
- added D49: LED_WS2812B, User_Footprints:LED_WS2812B_2x1.8mm, F.Cu at (176.1, 101.9)
- added D50: LED_WS2812B, User_Footprints:LED_WS2812B_2x1.8mm, F.Cu at (189.2, 121.8)
- added D51: LED_WS2812B, User_Footprints:LED_WS2812B_2x1.8mm, F.Cu at (176.1, 141.7)
- added D52: LED_WS2812B, User_Footprints:LED_WS2812B_2x1.8mm, F.Cu at (179.4, 101.9)
- added D53: LED_WS2812B, User_Footprints:LED_WS2812B_2x1.8mm, F.Cu at (185.9, 121.8)
- added D54: LED_WS2812B, User_Footprints:LED_WS2812B_2x1.8mm, F.Cu at (179.4, 141.7)
- added D55: LED_WS2812B, User_Footprints:LED_WS2812B_2x1.8mm, F.Cu at (186.0, 101.9)
- added D56: LED_WS2812B, User_Footprints:LED_WS2812B_2x1.8mm, F.Cu at (179.3, 121.8)
- added D62: LED_WS2812B, User_Footprints:LED_WS2812B_2x1.8mm, F.Cu at (192.6, 108.6)
- added D69: LED_WS2812B, User_Footprints:LED_WS2812B_2x1.8mm, F.Cu at (201.5, 105.3)
- added D90: LED_WS2812B, User_Footprints:LED_WS2812B_2x1.8mm, F.Cu at (221.4, 108.6)
- added J2: USB-C_Port, User_Footprints:GCT_USB4110GFA, F.Cu at (219.0, 154.0)
- added J3: TP4057, User_Footprints:SOT-23-6, F.Cu at (214.4, 150.7)
- added REF**: Fiducial_0.5mm_Mask1mm, Fiducial:Fiducial_0.5mm_Mask1mm, F.Cu at (92.0, 161.0)
- added REF**: Fiducial_0.5mm_Mask1mm, Fiducial:Fiducial_0.5mm_Mask1mm, F.Cu at (85.8, 148.2)
- added REF**: Fiducial_0.5mm_Mask1mm, Fiducial:Fiducial_0.5mm_Mask1mm, F.Cu at (204.8, 160.1)
- added REF**: Fiducial_0.5mm_Mask1mm, Fiducial:Fiducial_0.5mm_Mask1mm, F.Cu at (107.3, 148.9)
- added REF**: Fiducial_0.5mm_Mask1mm, Fiducial:Fiducial_0.5mm_Mask1mm, F.Cu at (216.4, 160.9)
- added REF**: Fiducial_0.5mm_Mask1mm, Fiducial:Fiducial_0.5mm_Mask1mm, F.Cu at (217.2, 146.7)
- added SW1: SW_Push, User_Footprints:Oval_Button, F.Cu at (196.6, 150.9)
- AE1: footprint User_Footprints:HM-NFC-Class6-Antenna -> User_Footprints:HM-NFC-Class3-Antenna
- BT1: value AA_BATTERY -> LiPo; footprint User_Footprints:BAT_BCAAPC -> User_Footprints:JST_PH_S2B-PH-K_1x02_P2.00mm_Horizontal
- BT2: value AA_BATTERY -> 18650_Cell; footprint User_Footprints:BAT_BCAAPC -> User_Footprints:18650_Cell_Holder
- BZ1: value HYG-9032A -> Buzzer; footprint User_Footprints:MagneticBuzzer_HYG-9032A -> User_Footprints:XDCR_CMT-7525-80-SMT-TR
- C1: value 10u -> 1u; footprint Capacitor_SMD:C_0603_1608Metric -> User_Footprints:C_0603_1608Metric
- C2: renamed from D37; value LED_RGAB -> 1u; footprint User_Footprints:RGB_LED_NH-B2020RGBA-HF -> User_Footprints:C_0603_1608Metric
- C3, C4: value 22u -> 18p; footprint Capacitor_SMD:C_0603_1608Metric -> User_Footprints:C_0603_1608Metric
- C5, C6: value 18p -> 4u7; footprint Capacitor_SMD:C_0603_1608Metric -> User_Footprints:C_0603_1608Metric
- D1: value LED_RGAB -> LED; footprint User_Footprints:RGB_LED_NH-B2020RGBA-HF -> LED_SMD:LED_0603_1608Metric
- D10, D100, D101, D102, D103, D104, D105, D106, D107, D108, D109, D11, D110, D111, D112, D113, D114, D115, D116, D117, D118, D119, D120, D121, D122, D123, D124, D125, D126, D127, D128, D129, D13, D130, D131, D132, D133, D134, D135, D136, D137, D138, D139, D14, D140, D141, D142, D143, D144, D145, D146, D147, D148, D149, D15, D150, D151, D152, D153, D154, D155, D156, D157, D158, D159, D16, D160, D161, D162, D163, D164, D165, D166, D167, D168, D17, D18, D19, D2, D20, D21, D22, D23, D24, D25, D26, D27, D28, D29, D3, D31, D32, D33, D34, D35, D36, D38, D39, D4, D5, D57, D58, D59, D60, D61, D63, D64, D65, D66, D67, D68, D7, D70, D71, D72, D73, D74, D75, D76, D77, D78, D79, D8, D80, D81, D82, D83, D84, D85, D86, D87, D88, D89, D9, D91, D92, D93, D94, D95, D96, D97, D98, D99: value LED_RGAB -> LED_WS2812B; footprint User_Footprints:RGB_LED_NH-B2020RGBA-HF -> User_Footprints:LED_WS2812B_2x1.8mm
- D12: renamed from D69; value LED_RGAB -> LED_WS2812B; footprint User_Footprints:RGB_LED_NH-B2020RGBA-HF -> User_Footprints:LED_WS2812B_2x1.8mm
- D30: renamed from D90; value LED_RGAB -> LED_WS2812B; footprint User_Footprints:RGB_LED_NH-B2020RGBA-HF -> User_Footprints:LED_WS2812B_2x1.8mm
- D6: renamed from D62; value LED_RGAB -> LED_WS2812B; footprint User_Footprints:RGB_LED_NH-B2020RGBA-HF -> User_Footprints:LED_WS2812B_2x1.8mm
- Q1, Q2, Q3, Q4: footprint Package_TO_SOT_SMD:SOT-23 -> User_Footprints:SOT-23
- R1, R2: footprint Resistor_SMD:R_0603_1608Metric -> User_Footprints:R_0603_1608Metric
- R10: value 12 -> 1K; footprint Resistor_SMD:R_1210_3225Metric -> User_Footprints:R_0603_1608Metric
- R11: value 15 -> 1K; footprint Resistor_SMD:R_1210_3225Metric -> User_Footprints:R_0603_1608Metric
- R12: value 62 -> 100K; footprint Resistor_SMD:R_0603_1608Metric -> User_Footprints:R_0603_1608Metric
- R13, R7: value 36 -> 100K; footprint Resistor_SMD:R_0603_1608Metric -> User_Footprints:R_0603_1608Metric
- R14: value 43 -> 100K; footprint Resistor_SMD:R_0603_1608Metric -> User_Footprints:R_0603_1608Metric
- R15: value 21 -> 1K; footprint Resistor_SMD:R_0603_1608Metric -> User_Footprints:R_0603_1608Metric
- R16, R18, R9: value 20 -> 1K; footprint Resistor_SMD:R_1210_3225Metric -> User_Footprints:R_0603_1608Metric
- R17: value 12 -> 1K; footprint Resistor_SMD:R_0603_1608Metric -> User_Footprints:R_0603_1608Metric
- R19: value 15 -> 1K; footprint Resistor_SMD:R_0603_1608Metric -> User_Footprints:R_0603_1608Metric
- R3: value 62 -> 1K; footprint Resistor_SMD:R_0603_1608Metric -> User_Footprints:R_0603_1608Metric
- R4: value 36 -> 1K6; footprint Resistor_SMD:R_0603_1608Metric -> User_Footprints:R_0603_1608Metric
- R5: value 43 -> 5K1; footprint Resistor_SMD:R_0603_1608Metric -> User_Footprints:R_0603_1608Metric
- R6: value 62 -> 5K1; footprint Resistor_SMD:R_0603_1608Metric -> User_Footprints:R_0603_1608Metric
- R8: value 43 -> 1K; footprint Resistor_SMD:R_0603_1608Metric -> User_Footprints:R_0603_1608Metric
- SW2, SW3: footprint User_Footprints:SW_SPST_TSC015A03526A -> User_Footprints:Oval_Button
- U1: value AP63203WU -> BC833M; footprint Package_TO_SOT_SMD:TSOT-23-6 -> User_Footprints:XCVR_BC833M
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Connections:
- BZ1 pad 1: Net-(U2-PadP$17) -> Net-(BZ1-Pad1)
- C1 pad 1: Net-(C1-Pad1) -> VBUS
- C2 pad 1: RED_BOTT_2 -> VBAT
- C2 pad 2: GREEN_BOTT_2 -> GND
- C3 pad 1: +3V3 -> Net-(AE1-Pad1)
- C4 pad 1: +3V3 -> GND
- C4 pad 2: GND -> Net-(AE1-Pad2)
- C5 pad 1: GND -> VBUS
- C5 pad 2: Net-(AE1-Pad2) -> GND
- C6 pad 1: Net-(AE1-Pad1) -> VDD
- D1 pad 1: RED_BOTT_1 -> Net-(D1-Pad1)
- D1 pad 2: unconnected-(D1-Pad2) -> Net-(D1-Pad2)
- D10 pad 1: RED_BOTT_2 -> VLEDS_E
- D10 pad 2: GREEN_BOTT_2 -> Net-(D10-Pad2)
- D10 pad 3: Segment_2-E_OUT -> GND
- D10 pad 4: BLUE_BOTT_2 -> Net-(D10-Pad4)
- D100 pad 1: RED_RIGHT_2 -> VLEDS
- D100 pad 2: GREEN_RIGHT_2 -> Net-(D100-Pad2)
- D100 pad 3: Segment_2-G_OUT -> GND
- D100 pad 4: BLUE_RIGHT_2 -> Net-(D100-Pad4)
- D101 pad 1: RED_RIGHT_2 -> VLEDS
- D101 pad 2: GREEN_RIGHT_2 -> Net-(D100-Pad4)
- D101 pad 3: Segment_2-A_OUT -> GND
- D101 pad 4: BLUE_RIGHT_2 -> Net-(D101-Pad4)
- D102 pad 1: RED_RIGHT_2 -> VLEDS
- D102 pad 2: GREEN_RIGHT_2 -> Net-(D101-Pad4)
- D102 pad 3: Segment_2-G_OUT -> GND
- D102 pad 4: BLUE_RIGHT_2 -> Net-(D102-Pad4)
- D103 pad 1: RED_RIGHT_2 -> VLEDS
- D103 pad 2: GREEN_RIGHT_2 -> Net-(D103-Pad2)
- D103 pad 3: Segment_2-D_OUT -> GND
- D103 pad 4: BLUE_RIGHT_2 -> Net-(D103-Pad4)
- D104 pad 1: RED_RIGHT_2 -> VLEDS
- D104 pad 2: GREEN_RIGHT_2 -> Net-(D103-Pad4)
- D104 pad 3: Segment_2-D_OUT -> GND
- D104 pad 4: BLUE_RIGHT_2 -> Net-(D104-Pad4)
- D105 pad 1: RED_RIGHT_2 -> VLEDS
- D105 pad 2: GREEN_RIGHT_2 -> Net-(D105-Pad2)
- D105 pad 3: Segment_2-B_OUT -> GND
- D105 pad 4: BLUE_RIGHT_2 -> Net-(D105-Pad4)
- D106 pad 1: RED_RIGHT_2 -> VLEDS
- D106 pad 2: GREEN_RIGHT_2 -> Net-(D106-Pad2)
- D106 pad 3: Segment_2-B_OUT -> GND
- D106 pad 4: BLUE_RIGHT_2 -> Net-(D106-Pad4)
- D107 pad 1: RED_RIGHT_2 -> VLEDS
- D107 pad 2: GREEN_RIGHT_2 -> Net-(D104-Pad4)
- D107 pad 3: Segment_2-C_OUT -> GND
- D107 pad 4: BLUE_RIGHT_2 -> Net-(D107-Pad4)
- D108 pad 1: RED_RIGHT_2 -> VLEDS
- D108 pad 2: GREEN_RIGHT_2 -> Net-(D108-Pad2)
- D108 pad 3: Segment_2-C_OUT -> GND
- D108 pad 4: BLUE_RIGHT_2 -> Net-(D105-Pad2)
- D109 pad 1: RED_RIGHT_2 -> VLEDS
- D109 pad 2: GREEN_RIGHT_2 -> Net-(D109-Pad2)
- D109 pad 3: Segment_2-B_OUT -> GND
- D109 pad 4: BLUE_RIGHT_2 -> Net-(D106-Pad2)
- D11 pad 1: RED_BOTT_1 -> VLEDS_E
- D11 pad 2: unconnected-(D11-Pad2) -> Net-(D11-Pad2)
- D11 pad 3: Segment_2-E_OUT -> GND
- D11 pad 4: unconnected-(D11-Pad4) -> Net-(D10-Pad2)
- D110 pad 1: RED_RIGHT_2 -> VLEDS
- D110 pad 2: GREEN_RIGHT_2 -> Net-(D107-Pad4)
- D110 pad 3: Segment_2-B_OUT -> GND
- D110 pad 4: BLUE_RIGHT_2 -> Net-(D110-Pad4)
- D111 pad 1: RED_RIGHT_2 -> VLEDS
- D111 pad 2: GREEN_RIGHT_2 -> Net-(D111-Pad2)
- D111 pad 3: Segment_2-C_OUT -> GND
- D111 pad 4: BLUE_RIGHT_2 -> Net-(D111-Pad4)
- D112 pad 1: RED_RIGHT_2 -> VLEDS
- D112 pad 2: GREEN_RIGHT_2 -> Net-(D112-Pad2)
- D112 pad 3: Segment_2-C_OUT -> GND
- D112 pad 4: BLUE_RIGHT_2 -> Net-(D112-Pad4)
- D113 pad 1: RED_LEFT_1 -> VLEDS
- D113 pad 2: GREEN_LEFT_1 -> Net-(D113-Pad2)
- D113 pad 3: Segment_2-F_OUT -> GND
- D113 pad 4: BLUE_LEFT_1 -> Net-(D113-Pad4)
- D114 pad 1: RED_LEFT_1 -> VLEDS
- D114 pad 2: GREEN_LEFT_1 -> Net-(D114-Pad2)
- D114 pad 3: Segment_2-F_OUT -> GND
- D114 pad 4: BLUE_LEFT_1 -> Net-(D111-Pad2)
- D115 pad 1: RED_LEFT_1 -> VLEDS
- D115 pad 2: GREEN_LEFT_1 -> unconnected-(D115-Pad2)
- D115 pad 3: Segment_2-E_OUT -> GND
- D115 pad 4: BLUE_LEFT_1 -> Net-(D112-Pad2)
- D116 pad 1: RED_LEFT_1 -> VLEDS
- D116 pad 2: GREEN_LEFT_1 -> Net-(D113-Pad4)
- D116 pad 3: Segment_2-E_OUT -> GND
- D116 pad 4: BLUE_LEFT_1 -> Net-(D116-Pad4)
- D117 pad 1: RED_LEFT_1 -> VLEDS
- D117 pad 2: GREEN_LEFT_1 -> Net-(D117-Pad2)
- D117 pad 3: Segment_2-F_OUT -> GND
- D117 pad 4: BLUE_LEFT_1 -> Net-(D117-Pad4)
- D118 pad 1: RED_LEFT_1 -> VLEDS
- D118 pad 2: GREEN_LEFT_1 -> Net-(D118-Pad2)
- D118 pad 3: Segment_2-F_OUT -> GND
- D118 pad 4: BLUE_LEFT_1 -> Net-(D117-Pad2)
- D119 pad 1: RED_LEFT_1 -> VLEDS
- D119 pad 2: GREEN_LEFT_1 -> Net-(D119-Pad2)
- D119 pad 3: Segment_2-E_OUT -> GND
- D119 pad 4: BLUE_LEFT_1 -> Net-(D119-Pad4)
- D12 pad 1: RED_RIGHT_1 -> VLEDS_E
- D12 pad 2: GREEN_RIGHT_1 -> unconnected-(D12-Pad2)
- D12 pad 3: Segment_2-D_OUT -> GND
- D12 pad 4: BLUE_RIGHT_1 -> Net-(D12-Pad4)
- D120 pad 1: RED_LEFT_1 -> VLEDS
- D120 pad 2: GREEN_LEFT_1 -> Net-(D106-Pad4)
- D120 pad 3: Segment_2-E_OUT -> GND
- D120 pad 4: BLUE_LEFT_1 -> Net-(D119-Pad2)
- D121 pad 1: RED_LEFT_1 -> VLEDS
- D121 pad 2: GREEN_LEFT_1 -> Net-(D121-Pad2)
- D121 pad 3: Segment_2-A_OUT -> GND
- D121 pad 4: BLUE_LEFT_1 -> L1_Data
- D122 pad 1: RED_LEFT_1 -> VLEDS
- D122 pad 2: GREEN_LEFT_1 -> Net-(D122-Pad2)
- D122 pad 3: Segment_2-G_OUT -> GND
- D122 pad 4: BLUE_LEFT_1 -> Net-(D121-Pad2)
- D123 pad 1: RED_LEFT_1 -> VLEDS
- D123 pad 2: GREEN_LEFT_1 -> Net-(D123-Pad2)
- D123 pad 3: Segment_2-A_OUT -> GND
- D123 pad 4: BLUE_LEFT_1 -> Net-(D123-Pad4)
- D124 pad 1: RED_LEFT_1 -> VLEDS
- D124 pad 2: GREEN_LEFT_1 -> Net-(D116-Pad4)
- D124 pad 3: Segment_2-G_OUT -> GND
- D124 pad 4: BLUE_LEFT_1 -> Net-(D123-Pad2)
- D125 pad 1: RED_LEFT_1 -> VLEDS
- D125 pad 2: GREEN_LEFT_1 -> Net-(D125-Pad2)
- D125 pad 3: Segment_2-D_OUT -> GND
- D125 pad 4: BLUE_LEFT_1 -> Net-(D125-Pad4)
- D126 pad 1: RED_LEFT_1 -> VLEDS
- D126 pad 2: GREEN_LEFT_1 -> Net-(D125-Pad4)
- D126 pad 3: Segment_2-D_OUT -> GND
- D126 pad 4: BLUE_LEFT_1 -> Net-(D126-Pad4)
- D127 pad 1: RED_LEFT_1 -> VLEDS
- D127 pad 2: GREEN_LEFT_1 -> Net-(D127-Pad2)
- D127 pad 3: Segment_2-A_OUT -> GND
- D127 pad 4: BLUE_LEFT_1 -> Net-(D127-Pad4)
- D128 pad 1: RED_LEFT_1 -> VLEDS
- D128 pad 2: GREEN_LEFT_1 -> Net-(D127-Pad4)
- D128 pad 3: Segment_2-G_OUT -> GND
- D128 pad 4: BLUE_LEFT_1 -> L2_Data
- D129 pad 1: RED_LEFT_1 -> VLEDS
- D129 pad 2: GREEN_LEFT_1 -> Net-(D129-Pad2)
- D129 pad 3: Segment_2-A_OUT -> GND
- D129 pad 4: BLUE_LEFT_1 -> Net-(D129-Pad4)
- D13 pad 1: unconnected-(D13-Pad1) -> VLEDS
- D13 pad 2: unconnected-(D13-Pad2) -> Net-(D13-Pad2)
- D13 pad 3: Segment_2-E_OUT -> GND
- D13 pad 4: BLUE_BOTT_1 -> Net-(D13-Pad4)
- D130 pad 1: RED_LEFT_1 -> VLEDS
- D130 pad 2: GREEN_LEFT_1 -> Net-(D129-Pad4)
- D130 pad 3: Segment_2-G_OUT -> GND
- D130 pad 4: BLUE_LEFT_1 -> Net-(D130-Pad4)
- D131 pad 1: RED_LEFT_1 -> VLEDS
- D131 pad 2: GREEN_LEFT_1 -> Net-(D131-Pad2)
- D131 pad 3: Segment_2-D_OUT -> GND
- D131 pad 4: BLUE_LEFT_1 -> Net-(D131-Pad4)
- D132 pad 1: RED_LEFT_1 -> VLEDS
- D132 pad 2: GREEN_LEFT_1 -> Net-(D131-Pad4)
- D132 pad 3: Segment_2-D_OUT -> GND
- D132 pad 4: BLUE_LEFT_1 -> Net-(D132-Pad4)
- D133 pad 1: RED_LEFT_1 -> VLEDS
- D133 pad 2: GREEN_LEFT_1 -> Net-(D133-Pad2)
- D133 pad 3: Segment_2-B_OUT -> GND
- D133 pad 4: BLUE_LEFT_1 -> Net-(D125-Pad2)
- D134 pad 1: RED_LEFT_1 -> VLEDS
- D134 pad 2: GREEN_LEFT_1 -> Net-(D134-Pad2)
- D134 pad 3: Segment_2-B_OUT -> GND
- D134 pad 4: BLUE_LEFT_1 -> Net-(D129-Pad2)
- D135 pad 1: RED_LEFT_1 -> VLEDS
- D135 pad 2: GREEN_LEFT_1 -> Net-(D132-Pad4)
- D135 pad 3: Segment_2-C_OUT -> GND
- D135 pad 4: BLUE_LEFT_1 -> Net-(D135-Pad4)
- D136 pad 1: RED_LEFT_1 -> VLEDS
- D136 pad 2: GREEN_LEFT_1 -> Net-(D136-Pad2)
- D136 pad 3: Segment_2-C_OUT -> GND
- D136 pad 4: BLUE_LEFT_1 -> Net-(D133-Pad2)
- D137 pad 1: RED_LEFT_1 -> VLEDS
- D137 pad 2: GREEN_LEFT_1 -> Net-(D137-Pad2)
- D137 pad 3: Segment_2-B_OUT -> GND
- D137 pad 4: BLUE_LEFT_1 -> Net-(D134-Pad2)
- D138 pad 1: RED_LEFT_1 -> VLEDS
- D138 pad 2: GREEN_LEFT_1 -> Net-(D135-Pad4)
- D138 pad 3: Segment_2-B_OUT -> GND
- D138 pad 4: BLUE_LEFT_1 -> Net-(D138-Pad4)
- D139 pad 1: RED_LEFT_1 -> VLEDS
- D139 pad 2: GREEN_LEFT_1 -> Net-(D139-Pad2)
- D139 pad 3: Segment_2-C_OUT -> GND
- D139 pad 4: BLUE_LEFT_1 -> Net-(D139-Pad4)
- D14 pad 1: RED_BOTT_2 -> VLEDS_E
- D14 pad 2: GREEN_BOTT_2 -> Net-(D10-Pad4)
- D14 pad 3: Segment_2-F_OUT -> GND
- D14 pad 4: BLUE_BOTT_2 -> Net-(D14-Pad4)
- D140 pad 1: RED_LEFT_1 -> VLEDS
- D140 pad 2: GREEN_LEFT_1 -> Net-(D140-Pad2)
- D140 pad 3: Segment_2-C_OUT -> GND
- D140 pad 4: BLUE_LEFT_1 -> Net-(D140-Pad4)
- D141 pad 1: RED_LEFT_2 -> VLEDS
- D141 pad 2: GREEN_LEFT_2 -> Net-(D141-Pad2)
- D141 pad 3: Segment_2-F_OUT -> GND
- D141 pad 4: BLUE_LEFT_2 -> Net-(D141-Pad4)
- D142 pad 1: RED_LEFT_2 -> VLEDS
- D142 pad 2: GREEN_LEFT_2 -> Net-(D142-Pad2)
- D142 pad 3: Segment_2-F_OUT -> GND
- D142 pad 4: BLUE_LEFT_2 -> Net-(D139-Pad2)
- D143 pad 1: RED_LEFT_2 -> VLEDS
- D143 pad 2: GREEN_LEFT_2 -> unconnected-(D143-Pad2)
- D143 pad 3: Segment_2-E_OUT -> GND
- D143 pad 4: BLUE_LEFT_2 -> Net-(D140-Pad2)
- D144 pad 1: RED_LEFT_2 -> VLEDS
- D144 pad 2: GREEN_LEFT_2 -> Net-(D141-Pad4)
- D144 pad 3: Segment_2-E_OUT -> GND
- D144 pad 4: BLUE_LEFT_2 -> Net-(D144-Pad4)
- D145 pad 1: RED_LEFT_2 -> VLEDS
- D145 pad 2: GREEN_LEFT_2 -> Net-(D145-Pad2)
- D145 pad 3: Segment_2-F_OUT -> GND
- D145 pad 4: BLUE_LEFT_2 -> Net-(D142-Pad2)
- D146 pad 1: RED_LEFT_2 -> VLEDS
- D146 pad 2: GREEN_LEFT_2 -> Net-(D146-Pad2)
- D146 pad 3: Segment_2-F_OUT -> GND
- D146 pad 4: BLUE_LEFT_2 -> Net-(D145-Pad2)
- D147 pad 1: RED_LEFT_2 -> VLEDS
- D147 pad 2: GREEN_LEFT_2 -> Net-(D147-Pad2)
- D147 pad 3: Segment_2-E_OUT -> GND
- D147 pad 4: BLUE_LEFT_2 -> Net-(D147-Pad4)
- D148 pad 1: RED_LEFT_2 -> VLEDS
- D148 pad 2: GREEN_LEFT_2 -> Net-(D148-Pad2)
- D148 pad 3: Segment_2-E_OUT -> GND
- D148 pad 4: BLUE_LEFT_2 -> Net-(D147-Pad2)
- D149 pad 1: RED_LEFT_2 -> VLEDS
- D149 pad 2: GREEN_LEFT_2 -> Net-(D149-Pad2)
- D149 pad 3: Segment_2-A_OUT -> GND
- D149 pad 4: BLUE_LEFT_2 -> Net-(D149-Pad4)
- D15 pad 1: RED_BOTT_2 -> VLEDS_E
- D15 pad 2: GREEN_BOTT_2 -> Net-(D12-Pad4)
- D15 pad 3: Segment_2-E_OUT -> GND
- D15 pad 4: BLUE_BOTT_2 -> Net-(D15-Pad4)
- D150 pad 1: RED_LEFT_2 -> VLEDS
- D150 pad 2: GREEN_LEFT_2 -> Net-(D150-Pad2)
- D150 pad 3: Segment_2-G_OUT -> GND
- D150 pad 4: BLUE_LEFT_2 -> Net-(D149-Pad2)
- D151 pad 1: RED_LEFT_2 -> VLEDS
- D151 pad 2: GREEN_LEFT_2 -> Net-(D151-Pad2)
- D151 pad 3: Segment_2-A_OUT -> GND
- D151 pad 4: BLUE_LEFT_2 -> Net-(D151-Pad4)
- D152 pad 1: RED_LEFT_2 -> VLEDS
- D152 pad 2: GREEN_LEFT_2 -> Net-(D144-Pad4)
- D152 pad 3: Segment_2-G_OUT -> GND
- D152 pad 4: BLUE_LEFT_2 -> Net-(D151-Pad2)
- D153 pad 1: RED_LEFT_2 -> VLEDS_E
- D153 pad 2: GREEN_LEFT_2 -> Net-(D153-Pad2)
- D153 pad 3: Segment_2-D_OUT -> GND
- D153 pad 4: BLUE_LEFT_2 -> Net-(D153-Pad4)
- D154 pad 1: RED_LEFT_2 -> VLEDS_E
- D154 pad 2: GREEN_LEFT_2 -> Net-(D154-Pad2)
- D154 pad 3: Segment_2-D_OUT -> GND
- D154 pad 4: BLUE_LEFT_2 -> Net-(D154-Pad4)
- D155 pad 1: RED_LEFT_2 -> VLEDS_E
- D155 pad 2: GREEN_LEFT_2 -> Net-(D155-Pad2)
- D155 pad 3: Segment_2-A_OUT -> GND
- D155 pad 4: BLUE_LEFT_2 -> Net-(D155-Pad4)
- D156 pad 1: RED_LEFT_2 -> VLEDS_E
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Routing:
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Other:
- outline, holes or cut-outs redrawn
- board text removed: "-"
- board text removed: "GND SWCLK GND SWDIO +3V3 SWO X X GND RST"
- board text removed: "Tag-Connect TC2050-IDC Programming Port"

Commit message: Created hardware revision 0.3, sent to fab.
Parts:
- removed BZ1: Buzzer, User_Footprints:XDCR_CMT-7525-80-SMT-TR
- removed Q1, Q2, Q3, Q4: HL-2301V, User_Footprints:SOT-23
- removed R10, R11, R15, R16, R17, R18, R19, R9: 1K, User_Footprints:R_0603_1608Metric
- removed R12, R13, R14: 100K, User_Footprints:R_0603_1608Metric
- removed REF** (x6): Fiducial_0.5mm_Mask1mm, Fiducial:Fiducial_0.5mm_Mask1mm
- added BZ2: Buzzer, User_Footprints:XDCR_CMT-7525-80-SMT-TR, F.Cu at (211.3, 156.8)
- added C10: 100n, Capacitor_SMD:C_0603_1608Metric, F.Cu at (207.4, 147.7)
- added C7: 100n, Capacitor_SMD:C_0603_1608Metric, F.Cu at (95.4, 148.9)
- added C8: 100n, Capacitor_SMD:C_0603_1608Metric, F.Cu at (97.5, 160.9)
- added C9: 1u, User_Footprints:C_0603_1608Metric, F.Cu at (95.5, 147.4)
- added Q5: HL-2302V, Package_TO_SOT_SMD:SOT-23, F.Cu at (205.1, 159.0)
- added Q6: HL-2302V, Package_TO_SOT_SMD:SOT-23, F.Cu at (205.1, 152.1)
- added Q7: HL-2302V, Package_TO_SOT_SMD:SOT-23, F.Cu at (205.1, 155.5)
- added R20: 1K, User_Footprints:R_0603_1608Metric, F.Cu at (216.3, 159.9)
- added R21: 100K, User_Footprints:R_0603_1608Metric, F.Cu at (202.4, 159.8)
- added R22: 1K, User_Footprints:R_0603_1608Metric, F.Cu at (202.4, 156.8)
- added R24: 21, User_Footprints:R_0603_1608Metric, F.Cu at (110.3, 151.2)
- added R25: 100, User_Footprints:R_0603_1608Metric, F.Cu at (208.3, 150.7)
- added R27: 21, User_Footprints:R_0603_1608Metric, F.Cu at (110.3, 152.7)
- added R28: 43, User_Footprints:R_0603_1608Metric, F.Cu at (110.3, 149.8)
- added R29: 43, User_Footprints:R_0603_1608Metric, F.Cu at (110.3, 154.2)
- added R46: 21, User_Footprints:R_0603_1608Metric, F.Cu at (110.3, 155.7)
- added R47: 43, User_Footprints:R_0603_1608Metric, F.Cu at (107.3, 157.1)
- added R48: 21, User_Footprints:R_0603_1608Metric, F.Cu at (107.1, 154.1)
- added R49: 21, User_Footprints:R_0603_1608Metric, F.Cu at (105.5, 157.2)
- added R50: 21, User_Footprints:R_0603_1608Metric, F.Cu at (105.5, 154.2)
- added R51: 43, User_Footprints:R_0603_1608Metric, F.Cu at (103.9, 157.2)
- added R58: 21, User_Footprints:R_0603_1608Metric, F.Cu at (103.9, 154.2)
- added R59: 21, User_Footprints:R_0603_1608Metric, F.Cu at (102.2, 157.1)
- added R60: 21, User_Footprints:R_0603_1608Metric, F.Cu at (102.3, 154.2)
- added R61: 43, User_Footprints:R_0603_1608Metric, F.Cu at (100.7, 157.1)
- added R62: 21, User_Footprints:R_0603_1608Metric, F.Cu at (100.6, 154.1)
- added U2: DW01A, Package_TO_SOT_SMD:SOT-23-6, F.Cu at (204.9, 148.3)
- added U3: IS31FL3729, Package_DFN_QFN:QFN-32-1EP_4x4mm_P0.4mm_EP2.9x2.9mm_ThermalVias, F.Cu at (105.5, 149.6)
- BT1: value LiPo -> LiPo_Plug
- BT2: value 18650_Cell -> 18650_Cell_Holder
- D10, D100, D101, D102, D103, D104, D105, D106, D107, D108, D109, D11, D110, D111, D112, D113, D114, D115, D116, D117, D118, D119, D12, D120, D121, D122, D123, D124, D125, D126, D127, D128, D129, D13, D130, D131, D132, D133, D134, D135, D136, D137, D138, D139, D14, D140, D141, D142, D143, D144, D145, D146, D147, D148, D149, D15, D150, D151, D152, D153, D154, D155, D156, D157, D158, D159, D16, D160, D161, D162, D163, D164, D165, D166, D167, D168, D169, D17, D170, D171, D172, D173, D174, D175, D176, D177, D178, D179, D18, D180, D181, D182, D183, D184, D19, D2, D20, D21, D22, D23, D24, D25, D26, D27, D28, D29, D3, D30, D31, D32, D33, D34, D35, D36, D37, D38, D39, D4, D40, D41, D42, D43, D44, D45, D46, D47, D48, D49, D5, D50, D51, D52, D53, D54, D55, D56, D57, D58, D59, D6, D60, D61, D62, D63, D64, D65, D66, D67, D68, D69, D7, D70, D71, D72, D73, D74, D75, D76, D77, D78, D79, D8, D80, D81, D82, D83, D84, D85, D86, D87, D88, D89, D9, D90, D91, D92, D93, D94, D95, D96, D97, D98, D99: value LED_WS2812B -> LED_RGAB; footprint User_Footprints:LED_WS2812B_2x1.8mm -> User_Footprints:RGB_LED_NH-B2020RGBA-HF
- J1: footprint User_Footprints:TC2050-IDC-FP -> User_Footprints:TAG-CONNECT_TC2050-IDC-NL
- R4: value 1K6 -> 5K1
- R5, R6: value 5K1 -> 2K
- R8: value 1K -> 10K
- SW1, SW2, SW3: footprint User_Footprints:Oval_Button -> User_Footprints:SW4_1437565_TEC
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Connections:
- BT1 pad 2: GND -> Net-(BT1--)
- BT2 pad 2: GND -> Net-(BT1--)
- D10 pad 1: VLEDS_E -> unconnected-(D10-RK-Pad1)
- D10 pad 2: Net-(D10-Pad2) -> unconnected-(D10-GK-Pad2)
- D10 pad 3: GND -> Segment_A
- D10 pad 4: Net-(D10-Pad4) -> GREEN_BOTTOM
- D100 pad 1: VLEDS -> RED_LEFT_1
- D100 pad 2: Net-(D100-Pad2) -> BLUE_LEFT_1
- D100 pad 3: GND -> Segment_F
- D100 pad 4: Net-(D100-Pad4) -> GREEN_LEFT_1
- D101 pad 1: VLEDS -> RED_LEFT_1
- D101 pad 2: Net-(D100-Pad4) -> BLUE_LEFT_1
- D101 pad 3: GND -> Segment_E
- D101 pad 4: Net-(D101-Pad4) -> GREEN_LEFT_1
- D102 pad 1: VLEDS -> RED_LEFT_1
- D102 pad 2: Net-(D101-Pad4) -> BLUE_LEFT_1
- D102 pad 3: GND -> Segment_E
- D102 pad 4: Net-(D102-Pad4) -> GREEN_LEFT_1
- D103 pad 1: VLEDS -> RED_LEFT_1
- D103 pad 2: Net-(D103-Pad2) -> BLUE_LEFT_1
- D103 pad 3: GND -> Segment_E
- D103 pad 4: Net-(D103-Pad4) -> GREEN_LEFT_1
- D104 pad 1: VLEDS -> RED_LEFT_1
- D104 pad 2: Net-(D103-Pad4) -> BLUE_LEFT_1
- D104 pad 3: GND -> Segment_E
- D104 pad 4: Net-(D104-Pad4) -> GREEN_LEFT_1
- D105 pad 1: VLEDS -> RED_LEFT_1
- D105 pad 2: Net-(D105-Pad2) -> BLUE_LEFT_1
- D105 pad 3: GND -> Segment_A
- D105 pad 4: Net-(D105-Pad4) -> GREEN_LEFT_1
- D106 pad 1: VLEDS -> RED_LEFT_1
- D106 pad 2: Net-(D106-Pad2) -> BLUE_LEFT_1
- D106 pad 3: GND -> Segment_G
- D106 pad 4: Net-(D106-Pad4) -> GREEN_LEFT_1
- D107 pad 1: VLEDS -> RED_LEFT_1
- D107 pad 2: Net-(D104-Pad4) -> BLUE_LEFT_1
- D107 pad 3: GND -> Segment_D
- D107 pad 4: Net-(D107-Pad4) -> GREEN_LEFT_1
- D108 pad 1: VLEDS -> RED_LEFT_1
- D108 pad 2: Net-(D108-Pad2) -> BLUE_LEFT_1
- D108 pad 3: GND -> Segment_A
- D108 pad 4: Net-(D105-Pad2) -> GREEN_LEFT_1
- D109 pad 1: VLEDS -> RED_LEFT_1
- D109 pad 2: Net-(D109-Pad2) -> BLUE_LEFT_1
- D109 pad 3: GND -> Segment_G
- D109 pad 4: Net-(D106-Pad2) -> GREEN_LEFT_1
- D11 pad 1: VLEDS_E -> RED_BOTTOM
- D11 pad 2: Net-(D11-Pad2) -> unconnected-(D11-GK-Pad2)
- D11 pad 3: GND -> Segment_A
- D11 pad 4: Net-(D10-Pad2) -> unconnected-(D11-BK-Pad4)
- D110 pad 1: VLEDS -> RED_LEFT_1
- D110 pad 2: Net-(D107-Pad4) -> BLUE_LEFT_1
- D110 pad 3: GND -> Segment_D
- D110 pad 4: Net-(D110-Pad4) -> GREEN_LEFT_1
- D111 pad 1: VLEDS -> RED_LEFT_1
- D111 pad 2: Net-(D111-Pad2) -> BLUE_LEFT_1
- D111 pad 3: GND -> Segment_A
- D111 pad 4: Net-(D111-Pad4) -> GREEN_LEFT_1
- D112 pad 1: VLEDS -> RED_LEFT_1
- D112 pad 2: Net-(D112-Pad2) -> BLUE_LEFT_1
- D112 pad 3: GND -> Segment_G
- D112 pad 4: Net-(D112-Pad4) -> GREEN_LEFT_1
- D113 pad 1: VLEDS -> RED_LEFT_1
- D113 pad 2: Net-(D113-Pad2) -> BLUE_LEFT_1
- D113 pad 3: GND -> Segment_D
- D113 pad 4: Net-(D113-Pad4) -> GREEN_LEFT_1
- D114 pad 1: VLEDS -> RED_LEFT_1
- D114 pad 2: Net-(D114-Pad2) -> BLUE_LEFT_1
- D114 pad 3: GND -> Segment_A
- D114 pad 4: Net-(D111-Pad2) -> GREEN_LEFT_1
- D115 pad 1: VLEDS -> RED_LEFT_1
- D115 pad 2: unconnected-(D115-Pad2) -> BLUE_LEFT_1
- D115 pad 3: GND -> Segment_G
- D115 pad 4: Net-(D112-Pad2) -> GREEN_LEFT_1
- D116 pad 1: VLEDS -> RED_LEFT_1
- D116 pad 2: Net-(D113-Pad4) -> BLUE_LEFT_1
- D116 pad 3: GND -> Segment_D
- D116 pad 4: Net-(D116-Pad4) -> GREEN_LEFT_1
- D117 pad 1: VLEDS -> RED_LEFT_1
- D117 pad 2: Net-(D117-Pad2) -> BLUE_LEFT_1
- D117 pad 3: GND -> Segment_B
- D117 pad 4: Net-(D117-Pad4) -> GREEN_LEFT_1
- D118 pad 1: VLEDS -> RED_LEFT_1
- D118 pad 2: Net-(D118-Pad2) -> BLUE_LEFT_1
- D118 pad 3: GND -> Segment_B
- D118 pad 4: Net-(D117-Pad2) -> GREEN_LEFT_1
- D119 pad 1: VLEDS -> RED_LEFT_1
- D119 pad 2: Net-(D119-Pad2) -> BLUE_LEFT_1
- D119 pad 3: GND -> Segment_B
- D119 pad 4: Net-(D119-Pad4) -> GREEN_LEFT_1
- D12 pad 1: VLEDS_E -> unconnected-(D12-RK-Pad1)
- D12 pad 2: unconnected-(D12-Pad2) -> BLUE_BOTTOM
- D12 pad 3: GND -> Segment_A
- D12 pad 4: Net-(D12-Pad4) -> unconnected-(D12-BK-Pad4)
- D120 pad 1: VLEDS -> RED_LEFT_1
- D120 pad 2: Net-(D106-Pad4) -> BLUE_LEFT_1
- D120 pad 3: GND -> Segment_B
- D120 pad 4: Net-(D119-Pad2) -> GREEN_LEFT_1
- D121 pad 1: VLEDS -> RED_LEFT_1
- D121 pad 2: Net-(D121-Pad2) -> BLUE_LEFT_1
- D121 pad 3: GND -> Segment_C
- D121 pad 4: L1_Data -> GREEN_LEFT_1
- D122 pad 1: VLEDS -> RED_LEFT_1
- D122 pad 2: Net-(D122-Pad2) -> BLUE_LEFT_1
- D122 pad 3: GND -> Segment_C
- D122 pad 4: Net-(D121-Pad2) -> GREEN_LEFT_1
- D123 pad 1: VLEDS -> RED_LEFT_1
- D123 pad 2: Net-(D123-Pad2) -> BLUE_LEFT_1
- D123 pad 3: GND -> Segment_C
- D123 pad 4: Net-(D123-Pad4) -> GREEN_LEFT_1
- D124 pad 1: VLEDS -> RED_LEFT_1
- D124 pad 2: Net-(D116-Pad4) -> BLUE_LEFT_1
- D124 pad 3: GND -> Segment_C
- D124 pad 4: Net-(D123-Pad2) -> GREEN_LEFT_1
- D125 pad 1: VLEDS -> RED_LEFT_2
- D125 pad 2: Net-(D125-Pad2) -> BLUE_LEFT_2
- D125 pad 3: GND -> Segment_F
- D125 pad 4: Net-(D125-Pad4) -> GREEN_LEFT_2
- D126 pad 1: VLEDS -> RED_LEFT_2
- D126 pad 2: Net-(D125-Pad4) -> BLUE_LEFT_2
- D126 pad 3: GND -> Segment_F
- D126 pad 4: Net-(D126-Pad4) -> GREEN_LEFT_2
- D127 pad 1: VLEDS -> RED_LEFT_2
- D127 pad 2: Net-(D127-Pad2) -> BLUE_LEFT_2
- D127 pad 3: GND -> Segment_F
- D127 pad 4: Net-(D127-Pad4) -> GREEN_LEFT_2
- D128 pad 1: VLEDS -> RED_LEFT_2
- D128 pad 2: Net-(D127-Pad4) -> BLUE_LEFT_2
- D128 pad 3: GND -> Segment_F
- D128 pad 4: L2_Data -> GREEN_LEFT_2
- D129 pad 1: VLEDS -> RED_LEFT_2
- D129 pad 2: Net-(D129-Pad2) -> BLUE_LEFT_2
- D129 pad 3: GND -> Segment_E
- D129 pad 4: Net-(D129-Pad4) -> GREEN_LEFT_2
- D13 pad 1: VLEDS -> RED_RIGHT_2
- D13 pad 2: Net-(D13-Pad2) -> BLUE_RIGHT_2
- D13 pad 3: GND -> Segment_I
- D13 pad 4: Net-(D13-Pad4) -> GREEN_RIGHT_2
- D130 pad 1: VLEDS -> RED_LEFT_2
- D130 pad 2: Net-(D129-Pad4) -> BLUE_LEFT_2
- D130 pad 3: GND -> Segment_E
- D130 pad 4: Net-(D130-Pad4) -> GREEN_LEFT_2
- D131 pad 1: VLEDS -> RED_LEFT_2
- D131 pad 2: Net-(D131-Pad2) -> BLUE_LEFT_2
- D131 pad 3: GND -> Segment_E
- D131 pad 4: Net-(D131-Pad4) -> GREEN_LEFT_2
- D132 pad 1: VLEDS -> RED_LEFT_2
- D132 pad 2: Net-(D131-Pad4) -> BLUE_LEFT_2
- D132 pad 3: GND -> Segment_E
- D132 pad 4: Net-(D132-Pad4) -> GREEN_LEFT_2
- D133 pad 1: VLEDS -> RED_LEFT_2
- D133 pad 2: Net-(D133-Pad2) -> BLUE_LEFT_2
- D133 pad 3: GND -> Segment_A
- D133 pad 4: Net-(D125-Pad2) -> GREEN_LEFT_2
- D134 pad 1: VLEDS -> RED_LEFT_2
- D134 pad 2: Net-(D134-Pad2) -> BLUE_LEFT_2
- D134 pad 3: GND -> Segment_G
- D134 pad 4: Net-(D129-Pad2) -> GREEN_LEFT_2
- D135 pad 1: VLEDS -> RED_LEFT_2
- D135 pad 2: Net-(D132-Pad4) -> BLUE_LEFT_2
- D135 pad 3: GND -> Segment_D
- D135 pad 4: Net-(D135-Pad4) -> GREEN_LEFT_2
- D136 pad 1: VLEDS -> RED_LEFT_2
- D136 pad 2: Net-(D136-Pad2) -> BLUE_LEFT_2
- D136 pad 3: GND -> Segment_A
- D136 pad 4: Net-(D133-Pad2) -> GREEN_LEFT_2
- D137 pad 1: VLEDS -> RED_LEFT_2
- D137 pad 2: Net-(D137-Pad2) -> BLUE_LEFT_2
- D137 pad 3: GND -> Segment_G
- D137 pad 4: Net-(D134-Pad2) -> GREEN_LEFT_2
- D138 pad 1: VLEDS -> RED_LEFT_2
- D138 pad 2: Net-(D135-Pad4) -> BLUE_LEFT_2
- D138 pad 3: GND -> Segment_D
- D138 pad 4: Net-(D138-Pad4) -> GREEN_LEFT_2
- D139 pad 1: VLEDS -> RED_LEFT_2
- D139 pad 2: Net-(D139-Pad2) -> BLUE_LEFT_2
- D139 pad 3: GND -> Segment_A
- D139 pad 4: Net-(D139-Pad4) -> GREEN_LEFT_2
- D14 pad 1: VLEDS_E -> unconnected-(D14-RK-Pad1)
- D14 pad 2: Net-(D10-Pad4) -> unconnected-(D14-GK-Pad2)
- D14 pad 3: GND -> Segment_B
- D14 pad 4: Net-(D14-Pad4) -> GREEN_BOTTOM
- D140 pad 1: VLEDS -> RED_LEFT_2
- D140 pad 2: Net-(D140-Pad2) -> BLUE_LEFT_2
- D140 pad 3: GND -> Segment_G
- D140 pad 4: Net-(D140-Pad4) -> GREEN_LEFT_2
- D141 pad 1: VLEDS -> RED_LEFT_2
- D141 pad 2: Net-(D141-Pad2) -> BLUE_LEFT_2
- D141 pad 3: GND -> Segment_D
- D141 pad 4: Net-(D141-Pad4) -> GREEN_LEFT_2
- D142 pad 1: VLEDS -> RED_LEFT_2
- D142 pad 2: Net-(D142-Pad2) -> BLUE_LEFT_2
- D142 pad 3: GND -> Segment_A
- D142 pad 4: Net-(D139-Pad2) -> GREEN_LEFT_2
- D143 pad 1: VLEDS -> RED_LEFT_2
- D143 pad 2: unconnected-(D143-Pad2) -> BLUE_LEFT_2
- D143 pad 3: GND -> Segment_G
- D143 pad 4: Net-(D140-Pad2) -> GREEN_LEFT_2
- D144 pad 1: VLEDS -> RED_LEFT_2
- D144 pad 2: Net-(D141-Pad4) -> BLUE_LEFT_2
- D144 pad 3: GND -> Segment_D
- D144 pad 4: Net-(D144-Pad4) -> GREEN_LEFT_2
- D145 pad 1: VLEDS -> RED_LEFT_2
- D145 pad 2: Net-(D145-Pad2) -> BLUE_LEFT_2
- D145 pad 3: GND -> Segment_B
- D145 pad 4: Net-(D142-Pad2) -> GREEN_LEFT_2
- D146 pad 1: VLEDS -> RED_LEFT_2
- D146 pad 2: Net-(D146-Pad2) -> BLUE_LEFT_2
- D146 pad 3: GND -> Segment_B
- D146 pad 4: Net-(D145-Pad2) -> GREEN_LEFT_2
- D147 pad 1: VLEDS -> RED_LEFT_2
- D147 pad 2: Net-(D147-Pad2) -> BLUE_LEFT_2
- D147 pad 3: GND -> Segment_B
- D147 pad 4: Net-(D147-Pad4) -> GREEN_LEFT_2
- D148 pad 1: VLEDS -> RED_LEFT_2
- D148 pad 2: Net-(D148-Pad2) -> BLUE_LEFT_2
- D148 pad 3: GND -> Segment_B
- D148 pad 4: Net-(D147-Pad2) -> GREEN_LEFT_2
- D149 pad 1: VLEDS -> RED_LEFT_2
- D149 pad 2: Net-(D149-Pad2) -> BLUE_LEFT_2
- D149 pad 3: GND -> Segment_C
- D149 pad 4: Net-(D149-Pad4) -> GREEN_LEFT_2
- D15 pad 1: VLEDS_E -> unconnected-(D15-RK-Pad1)
- D15 pad 2: Net-(D12-Pad4) -> BLUE_BOTTOM
- D15 pad 3: GND -> Segment_B
- D15 pad 4: Net-(D15-Pad4) -> unconnected-(D15-BK-Pad4)
- D150 pad 1: VLEDS -> RED_LEFT_2
- D150 pad 2: Net-(D150-Pad2) -> BLUE_LEFT_2
- D150 pad 3: GND -> Segment_C
- D150 pad 4: Net-(D149-Pad2) -> GREEN_LEFT_2
- D151 pad 1: VLEDS -> RED_LEFT_2
- D151 pad 2: Net-(D151-Pad2) -> BLUE_LEFT_2
- D151 pad 3: GND -> Segment_C
- D151 pad 4: Net-(D151-Pad4) -> GREEN_LEFT_2
- D152 pad 1: VLEDS -> RED_LEFT_2
- D152 pad 2: Net-(D144-Pad4) -> BLUE_LEFT_2
- D152 pad 3: GND -> Segment_C
- D152 pad 4: Net-(D151-Pad2) -> GREEN_LEFT_2
- D153 pad 1: VLEDS_E -> RED_LEFT_1
- D153 pad 2: Net-(D153-Pad2) -> BLUE_LEFT_1
- D153 pad 3: GND -> Segment_I
- D153 pad 4: Net-(D153-Pad4) -> GREEN_LEFT_1
- D154 pad 1: VLEDS_E -> RED_LEFT_1
- D154 pad 2: Net-(D154-Pad2) -> BLUE_LEFT_1
- D154 pad 3: GND -> Segment_H
- D154 pad 4: Net-(D154-Pad4) -> GREEN_LEFT_1
- D155 pad 1: VLEDS_E -> RED_RIGHT_1
- D155 pad 2: Net-(D155-Pad2) -> BLUE_RIGHT_1
- D155 pad 3: GND -> Segment_I
- D155 pad 4: Net-(D155-Pad4) -> GREEN_RIGHT_1
- D156 pad 1: VLEDS_E -> RED_RIGHT_1
- D156 pad 2: Net-(D156-Pad2) -> BLUE_RIGHT_1
- D156 pad 3: GND -> Segment_H
- D156 pad 4: Net-(D156-Pad4) -> GREEN_RIGHT_1
- D157 pad 1: VLEDS -> RED_RIGHT_1
- D157 pad 2: Net-(D157-Pad2) -> BLUE_RIGHT_1
- D157 pad 3: GND -> Segment_F
- D157 pad 4: Net-(D157-Pad4) -> GREEN_RIGHT_1
- D158 pad 1: VLEDS -> RED_RIGHT_1
- D158 pad 2: Net-(D158-Pad2) -> BLUE_RIGHT_1
- D158 pad 3: GND -> Segment_E
- D158 pad 4: Net-(D158-Pad4) -> GREEN_RIGHT_1
- D159 pad 1: VLEDS -> RED_RIGHT_1
- D159 pad 2: Net-(D159-Pad2) -> BLUE_RIGHT_1
- D159 pad 3: GND -> Segment_A
- D159 pad 4: Net-(D159-Pad4) -> GREEN_RIGHT_1
- D16 pad 1: VLEDS_E -> RED_BOTTOM
- D16 pad 2: Net-(D16-Pad2) -> unconnected-(D16-GK-Pad2)
- D16 pad 3: GND -> Segment_B
- D16 pad 4: Net-(D11-Pad2) -> unconnected-(D16-BK-Pad4)
- D160 pad 1: VLEDS -> RED_RIGHT_1
- D160 pad 2: Net-(D160-Pad2) -> BLUE_RIGHT_1
- D160 pad 3: GND -> Segment_G
- D160 pad 4: Net-(D160-Pad4) -> GREEN_RIGHT_1
- D161 pad 1: VLEDS -> RED_RIGHT_1
- D161 pad 2: Net-(D161-Pad2) -> BLUE_RIGHT_1
- D161 pad 3: GND -> Segment_D
- D161 pad 4: Net-(D161-Pad4) -> GREEN_RIGHT_1
- D162 pad 1: VLEDS -> RED_RIGHT_1
- D162 pad 2: Net-(D162-Pad2) -> BLUE_RIGHT_1
- D162 pad 3: GND -> Segment_B
- D162 pad 4: Net-(D162-Pad4) -> GREEN_RIGHT_1
- D163 pad 1: VLEDS -> RED_RIGHT_1
- D163 pad 2: Net-(D163-Pad2) -> BLUE_RIGHT_1
- D163 pad 3: GND -> Segment_C
- D163 pad 4: Net-(D163-Pad4) -> GREEN_RIGHT_1
- D164 pad 1: VLEDS -> RED_RIGHT_2
- D164 pad 2: Net-(D164-Pad2) -> BLUE_RIGHT_2
- D164 pad 3: GND -> Segment_F
- D164 pad 4: Net-(D164-Pad4) -> GREEN_RIGHT_2
- D165 pad 1: VLEDS -> RED_RIGHT_2
- D165 pad 2: Net-(D165-Pad2) -> BLUE_RIGHT_2
- D165 pad 3: GND -> Segment_E
- D165 pad 4: Net-(D165-Pad4) -> GREEN_RIGHT_2
- D166 pad 1: VLEDS -> RED_RIGHT_2
- D166 pad 2: Net-(D166-Pad2) -> BLUE_RIGHT_2
- D166 pad 3: GND -> Segment_A
- D166 pad 4: Net-(D166-Pad4) -> GREEN_RIGHT_2
- D167 pad 1: VLEDS -> RED_RIGHT_2
- D167 pad 2: Net-(D167-Pad2) -> BLUE_RIGHT_2
- D167 pad 3: GND -> Segment_G
- D167 pad 4: Net-(D167-Pad4) -> GREEN_RIGHT_2
- D168 pad 1: VLEDS -> RED_RIGHT_2
- D168 pad 2: Net-(D168-Pad2) -> BLUE_RIGHT_2
- D168 pad 3: GND -> Segment_D
- D168 pad 4: Net-(D168-Pad4) -> GREEN_RIGHT_2
- D169 pad 1: VLEDS -> RED_RIGHT_2
- D169 pad 2: Net-(D169-Pad2) -> BLUE_RIGHT_2
- D169 pad 3: GND -> Segment_B
- D169 pad 4: Net-(D169-Pad4) -> GREEN_RIGHT_2
- D17 pad 1: VLEDS_E -> RED_RIGHT_2
- D17 pad 2: Net-(D17-Pad2) -> BLUE_RIGHT_2
- D17 pad 3: GND -> Segment_H
- D17 pad 4: Net-(D17-Pad4) -> GREEN_RIGHT_2
- D170 pad 1: VLEDS -> RED_RIGHT_2
- D170 pad 2: Net-(D170-Pad2) -> BLUE_RIGHT_2
- D170 pad 3: GND -> Segment_C
- D170 pad 4: Net-(D170-Pad4) -> GREEN_RIGHT_2
- D171 pad 1: VLEDS -> RED_LEFT_1
- D171 pad 2: Net-(D171-Pad2) -> BLUE_LEFT_1
- D171 pad 3: GND -> Segment_F
- D171 pad 4: Net-(D171-Pad4) -> GREEN_LEFT_1
- D172 pad 1: VLEDS -> RED_LEFT_1
- D172 pad 2: Net-(D102-Pad4) -> BLUE_LEFT_1
- D172 pad 3: GND -> Segment_E
- D172 pad 4: Net-(D103-Pad2) -> GREEN_LEFT_1
- D173 pad 1: VLEDS -> RED_LEFT_1
- D173 pad 2: Net-(D111-Pad4) -> BLUE_LEFT_1
- D173 pad 3: GND -> Segment_A
- D173 pad 4: Net-(D108-Pad2) -> GREEN_LEFT_1
- D174 pad 1: VLEDS -> RED_LEFT_1
- D174 pad 2: Net-(D112-Pad4) -> BLUE_LEFT_1
- D174 pad 3: GND -> Segment_G
- D174 pad 4: Net-(D109-Pad2) -> GREEN_LEFT_1
- D175 pad 1: VLEDS -> RED_LEFT_1
- D175 pad 2: Net-(D110-Pad4) -> BLUE_LEFT_1
- D175 pad 3: GND -> Segment_D
- D175 pad 4: Net-(D113-Pad2) -> GREEN_LEFT_1
- D176 pad 1: VLEDS -> RED_LEFT_1
- D176 pad 2: Net-(D119-Pad4) -> BLUE_LEFT_1
- D176 pad 3: GND -> Segment_B
- D176 pad 4: Net-(D118-Pad2) -> GREEN_LEFT_1
- D177 pad 1: VLEDS -> RED_LEFT_1
- D177 pad 2: Net-(D123-Pad4) -> BLUE_LEFT_1
- D177 pad 3: GND -> Segment_C
- D177 pad 4: Net-(D122-Pad2) -> GREEN_LEFT_1
- D178 pad 1: VLEDS -> RED_LEFT_2
- D178 pad 2: Net-(D126-Pad4) -> BLUE_LEFT_2
- D178 pad 3: GND -> Segment_F
- D178 pad 4: Net-(D127-Pad2) -> GREEN_LEFT_2
- D179 pad 1: VLEDS -> RED_LEFT_2
- D179 pad 2: Net-(D130-Pad4) -> BLUE_LEFT_2
- D179 pad 3: GND -> Segment_E
- D179 pad 4: Net-(D131-Pad2) -> GREEN_LEFT_2
- D18 pad 1: VLEDS_E -> unconnected-(D18-RK-Pad1)
- D18 pad 2: Net-(D14-Pad4) -> unconnected-(D18-GK-Pad2)
- D18 pad 3: GND -> Segment_C
- D18 pad 4: Net-(D18-Pad4) -> GREEN_BOTTOM
- D180 pad 1: VLEDS -> RED_LEFT_2
- D180 pad 2: Net-(D139-Pad4) -> BLUE_LEFT_2
- D180 pad 3: GND -> Segment_A
- D180 pad 4: Net-(D136-Pad2) -> GREEN_LEFT_2
- D181 pad 1: VLEDS -> RED_LEFT_2
- D181 pad 2: Net-(D140-Pad4) -> BLUE_LEFT_2
- D181 pad 3: GND -> Segment_G
- D181 pad 4: Net-(D137-Pad2) -> GREEN_LEFT_2
- D182 pad 1: VLEDS -> RED_LEFT_2
- D182 pad 2: Net-(D138-Pad4) -> BLUE_LEFT_2
- D182 pad 3: GND -> Segment_D
- D182 pad 4: Net-(D141-Pad2) -> GREEN_LEFT_2
- D183 pad 1: VLEDS -> RED_LEFT_2
- D183 pad 2: Net-(D147-Pad4) -> BLUE_LEFT_2
- D183 pad 3: GND -> Segment_B
- D183 pad 4: Net-(D146-Pad2) -> GREEN_LEFT_2
- D184 pad 1: VLEDS -> RED_LEFT_2
- D184 pad 2: Net-(D151-Pad4) -> BLUE_LEFT_2
- D184 pad 3: GND -> Segment_C
- D184 pad 4: Net-(D150-Pad2) -> GREEN_LEFT_2
- D19 pad 1: VLEDS_E -> unconnected-(D19-RK-Pad1)
- D19 pad 2: Net-(D15-Pad4) -> BLUE_BOTTOM
- D19 pad 3: GND -> Segment_C
- D19 pad 4: Net-(D19-Pad4) -> unconnected-(D19-BK-Pad4)
- D2 pad 1: VLEDS_E -> RED_LEFT_1
- D2 pad 2: Net-(D17-Pad4) -> BLUE_LEFT_1
- D2 pad 3: GND -> Segment_I
- D2 pad 4: Net-(D2-Pad4) -> GREEN_LEFT_1
- D20 pad 1: VLEDS -> RED_LEFT_2
- D20 pad 2: Net-(D117-Pad4) -> BLUE_LEFT_2
- D20 pad 3: GND -> Segment_I
- D20 pad 4: Net-(D114-Pad2) -> GREEN_LEFT_2
- D21 pad 1: VLEDS -> RED_LEFT_2
- D21 pad 2: Net-(D21-Pad2) -> BLUE_LEFT_2
- D21 pad 3: GND -> Segment_H
- D21 pad 4: Net-(D148-Pad2) -> GREEN_LEFT_2
- D22 pad 1: VLEDS_E -> RED_BOTTOM
- D22 pad 2: Net-(D22-Pad2) -> unconnected-(D22-GK-Pad2)
- D22 pad 3: GND -> Segment_C
- D22 pad 4: Net-(D16-Pad2) -> unconnected-(D22-BK-Pad4)
- D23 pad 1: VLEDS_E -> unconnected-(D23-RK-Pad1)
- D23 pad 2: Net-(D18-Pad4) -> unconnected-(D23-GK-Pad2)
- D23 pad 3: GND -> Segment_D
- D23 pad 4: Net-(D23-Pad4) -> GREEN_BOTTOM
- D24 pad 1: VLEDS_E -> unconnected-(D24-RK-Pad1)
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Routing:
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- added copper zone on B.Cu, net GND

Commit message: Fixed missing ground connection
Connections:
- J3 pad 5: Net-(J3-STDBY) -> GND
- R4 pad 2: Net-(J3-STDBY) -> GND
Routing:
- net GND: track 330.8 -> 337.1 mm
- net Net-(J3-STDBY): track 5.17 -> 0.00 mm
