File: Scoreboard.kicad_sch (KiCad schematic)
At the start: 39 parts, among them J1 TC2050-IDC-NL, P1 USB_C_Plug_USB2.0, Q1 HL-2301V, Q2 HL-2301V, Q3 HL-2301V, Q4 HL-2301V, Q5 HL-2301V, Q6 HL-2301V, Q7 HL-2301V, SW2 SW_Push, SW3 SW_Push, SW4 SW_Push, U1 AP63203WU, U2 BM832, U3 LM66100DCKR, U4 LM66100DCKR

Commit message: Made a new hardware revision
Parts:
- removed BT1, BT2, BT3: AA_BATTERY, User_Footprints:BAT_BCAAPC, symbol User_Symbols:AA_BATTERY
- removed C7: 1u, Capacitor_SMD:C_0603_1608Metric, symbol Device:C
- removed C8: 4u7, Capacitor_SMD:C_0603_1608Metric, symbol Device:C
- removed L1: 4u7, Inductor_SMD:L_0603_1608Metric, symbol Device:L
- removed P1: USB_C_Plug_USB2.0, User_Footprints:DEALON_USB-TYPE-C-009, symbol User_Symbols:USB_C_Plug_USB2.0
- removed Q5, Q6, Q7: HL-2301V, Package_TO_SOT_SMD:SOT-23, symbol User_Symbols:HL-2301V
- removed R33, R34, R35, R36, R37, R38, R39: 1K, Resistor_SMD:R_0603_1608Metric, symbol Device:R
- removed SW4: SW_Push, User_Footprints:SW_SPST_TSC015A03526A, symbol Switch:SW_Push
- removed U1: AP63203WU, Package_TO_SOT_SMD:TSOT-23-6, symbol Regulator_Switching:AP63203WU
- removed U2: BM832, User_Footprints:BM832, symbol User_Symbols:BM832
- removed U3, U4: LM66100DCKR, User_Footprints:DCK6_TEX-L, symbol User_Symbols:LM66100DCKR
- added BT1, BT2: (no value), symbol Device:Battery_Cell
- added D1: (no value), symbol Device:LED
- added J2: (no value), symbol User_Symbols:USB-C_Port
- added J3: (no value), symbol User_Symbols:TP4057
- added R10, R11, R12, R13, R14, R15, R16, R17, R18, R19, R3, R4, R5, R6, R7, R8, R9: (no value), symbol Device:R
- added SW1: (no value), symbol Switch:SW_Push
- added U1: (no value), symbol User_Symbols:BC833M
- AE1: value Antenna_Loop -> (none); footprint User_Footprints:HM-NFC-Class6-Antenna -> (none)
- BZ1: value HYG-9032A -> (none); footprint User_Footprints:MagneticBuzzer_HYG-9032A -> (none); Manufacturer HYDZ -> KELIKING; Notes 2.5-4.5V 85dB -> 2-4.5V 85dB 2.731kHz; Part Number HYG-9032A -> KLJ-7525-3627; Price .1835 -> .4741; Website https://www.lcsc.com/product-detail/Buzzers_HYDZ-HYG-9032A_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 -> https://www.lcsc.com/product-detail/Buzzers_KELIKING-KLJ-75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
- C1: value 10u -> (none); footprint Capacitor_SMD:C_0603_1608Metric -> (none); Notes 6.3V 20% -> 16V 10%; Part Number CL10A106MQ8NNNC -> CL10A105KO8NNNC; Price .0045 -> .0032; Website https://www.lcsc.com/product-detail/Multilayer-Ceramic-Capacitors-MLCC-SMD-SMT_Samsung-Electro-Mechanics-CL10A106MQ8NNNC_C1691.html -> https://www.lcsc.com/product-detail/Multilayer-Ceramic-Capacitors-MLCC-SMD-SMT_Samsung-Electro-Mechanics-CL10A105KO8NNNC_C1592.html
- C2: value 100n -> (none); footprint Capacitor_SMD:C_0603_1608Metric -> (none); Notes 25V 10% -> 16V 10%; Part Number CL10B104KA8NNNC -> CL10A105KO8NNNC; Price .0028 -> .0032; Website https://www.lcsc.com/product-detail/Multilayer-Ceramic-Capacitors-MLCC-SMD-SMT_Samsung-Electro-Mechanics-CL10B104KA8NNNC_C1590.html -> https://www.lcsc.com/product-detail/Multilayer-Ceramic-Capacitors-MLCC-SMD-SMT_Samsung-Electro-Mechanics-CL10A105KO8NNNC_C1592.html
- C3, C4: value 22u -> (none); footprint Capacitor_SMD:C_0603_1608Metric -> (none); Manufacturer Samsung Electro-Mechanics -> FOJAN; Notes 6.3V 20% -> 50V 5%; Part Number CL10A226MQ8NRNE -> FCC0603N180J500CT; Price .0098 -> .0027; Website https://www.lcsc.com/product-detail/Multilayer-Ceramic-Capacitors-MLCC-SMD-SMT_Samsung-Electro-Mechanics-CL10A226MQ8NRNE_C159801.html -> https://www.lcsc.com/product-detail/Multilayer-Ceramic-Capacitors-MLCC-SMD-SMT_FOJAN-FCC0603N180J500CT_C5137620.html
- C5, C6: value 18p -> (none); footprint Capacitor_SMD:C_0603_1608Metric -> (none); Manufacturer FOJAN -> HRE; Notes 50V 5% -> 6.3V 10%; Part Number FCC0603N180J500CT -> CSA0603X5R475K6R3JT; Price .0027 -> .0050; Website https://www.lcsc.com/product-detail/Multilayer-Ceramic-Capacitors-MLCC-SMD-SMT_FOJAN-FCC0603N180J500CT_C5137620.html -> https://www.lcsc.com/product-detail/Multilayer-Ceramic-Capacitors-MLCC-SMD-SMT_HRE-CSA0603X5R475K6R3JT_C3015159.html
- J1: value TC2050-IDC-NL -> (none); footprint User_Footprints:TC2050-IDC-FP -> (none)
- Q1, Q2, Q3, Q4: value HL-2301V -> (none); footprint Package_TO_SOT_SMD:SOT-23 -> (none)
- R1, R2: value 5K1 -> (none); footprint Resistor_SMD:R_0603_1608Metric -> (none)
- SW2, SW3: value SW_Push -> (none); footprint User_Footprints:SW_SPST_TSC015A03526A -> (none); Part Number TSC015A03526A -> TSA016A2526A; Price .0098 -> .0136; Website https://www.lcsc.com/product-detail/Tactile-Switches_BZCN-TSC015A03526A_C2888900.html -> https://www.lcsc.com/product-detail/Tactile-Switches_BZCN-TSA016A2526A_C2888428.html
Connections:
- net Segment_2-D_OUT is gone; now on an unnamed net: Q4.3 (D)
- net GND: now also C2.2, C4.1, C5.2, R2.2, BT1.2 (-), BT2.2 (-), J2.A1/B12 (GND), J2.B1/A12 (GND__1), J2.S1 (GND__2), J2.S2 (GND__3), J2.S3 (GND__4), J2.S4 (GND__5), J3.2 (GND), J3.5 (STDBY), R4.2, R6.2, SW1.1, U1.05 (GND), U1.25 (GND), U1.26 (GND), U1.27 (GND), U1.28 (GND); no longer C4.2, C5.1, R2.1
- net RST: now also U1.08 (P031)
- net SWCLK: now also U1.22 (SWDCLK)
- net SWDIO: now also U1.18 (SWDIO)
- net VBAT: now reaches C2.1
- net VBAT: now also Q1.2 (S), BT1.1 (+), BT2.1 (+), J3.3 (BAT)
- net at SW3.2: now also U1.21 (P020)
- net at AE1.2: now also C4.2, U1.23 (P009); no longer C5.2
- net at AE1.1: now also C3.1, U1.24 (P010); no longer C6.1
- net VBUS: now reaches C1.1
- net VBUS: now also C5.1, Q2.2 (S), Q3.2 (S), Q4.2 (S), J2.A4/B9 (VBUS), J2.B4/A9 (VBUS__1), J3.4 (VCC), R3.1, U1.13 (VDDH), U1.14 (VBUS)
- net at R1.1: now also J2.A5 (CC1)
- net at Q1.1 (G): now also R7.2, R8.2
- net at Q4.1 (G): now also R11.2, R14.2
- net at Q2.1 (G): now also R12.2, R9.2
- net at Q3.1 (G): now also R10.2, R13.2
- removed net +3V3: C3.1, C4.1, J1.1 (VTref), Q1.2 (S), Q2.2 (S), Q3.2 (S), Q4.2 (S)
- net SWO: no longer names the net of SW2.2
- net SWO: now also U1.17 (P018); no longer J1.6 (SWO/TDO)
- net Segment_2-A_OUT: no longer names the net of Q1.3 (D)
- net Segment_2-A_OUT: now also R5.1
- net Segment_2-B_OUT renamed VLEDS
- net Segment_2-C_OUT renamed VLEDS_E
- new net: D1.1 (K), J3.1 (CHG)
- new net: D1.2 (A), R3.2
- new net: R8.1, U1.07 (P030)
- new net: R5.2, R6.1, U1.02 (P003)
- new net: R11.1, U1.03 (P002)
- new net: R9.1, U1.04 (P028)
- new net: R10.1, U1.06 (P029)
- new net: R15.2, U1.09 (P004)
- new net: R16.2, U1.10 (P005)
- new net: R19.1, U1.11 (P109)
- new net: R17.2, U1.12 (P011)
- new net: R18.2, U1.16 (P015)
- new net: SW1.2, U1.20 (P017)
- new net: J2.B5 (CC2), R2.1
- new net: J3.6 (PROG), R4.1
- new net D+: J2.A6 (DP1), J2.B6 (DP2), U1.15 (D-)
- new net D-: J2.A7 (DN1), J2.B7 (DN2), U1.19 (D+)
- new net E1_Data: R18.1
- new net L1_Data: R17.1
- new net L2_Data: R19.2
- new net R1_Data: R16.1
- new net R2_Data: R15.1
- new net VDD: C6.1, J1.1 (VTref), R12.1, R13.1, R14.1, R7.1, U1.01 (VDD)
- no-connect marks 2 -> 5
Other:
- sheet Bottom_Display ports: added E1_DIN, E_VDD, E_VSS; removed BLUE_BOTT, BLUE_BOTT2, GREEN_BOTT, GREEN_BOTT2, RED_BOTT, RED_BOTT2, Segment_2-A, Segment_2-B, Segment_2-C, Segment_2-D, Segment_2-E, Segment_2-F, Segment_2-G
- sheet Left_Display ports: added L1_DIN, L2_DIN, L_VDD, L_VSS; removed BLUE_LEFT1, BLUE_LEFT2, GREEN_LEFT1, GREEN_LEFT2, RED_LEFT1, RED_LEFT2, Segment_2-A, Segment_2-B, Segment_2-C, Segment_2-D, Segment_2-E, Segment_2-F, Segment_2-G
- sheet Right_Display ports: added R1_DIN, R2_DIN, R_VDD, R_VSS; removed BLUE_RIGHT, BLUE_RIGHT2, GREEN_RIGHT, GREEN_RIGHT2, RED_RIGHT, RED_RIGHT2, Segment_2-A, Segment_2-B, Segment_2-C, Segment_2-D, Segment_2-E, Segment_2-F, Segment_2-G
- moved on the sheet: J1

Commit message: new version with indexed leds
Parts:
- AE1: value (none) -> Antenna_Loop; footprint (none) -> User_Footprints:HM-NFC-Class3-Antenna; Manufacturer (none) -> N/a; Notes (none) -> Integrated; Package (none) -> N/a; now not fitted; now in the parts list
- BT1: value (none) -> LiPo_Plug; footprint (none) -> User_Footprints:JST_PH_S2B-PH-K_1x02_P2.00mm_Horizontal; Manufacturer (none) -> XUNPU; Notes (none) -> 2A; Package (none) -> SMD 2mm P; Part Number (none) -> WAFER-PH2.0-2PWB; Price (none) -> .048; Vendor (none) -> LCSC; now not fitted
- BT2: value (none) -> 18650_Cell_Holder; footprint (none) -> User_Footprints:18650_Cell_Holder; Manufacturer (none) -> MYOUNG; Package (none) -> THT; Part Number (none) -> BH-18650-A1AJ005; Vendor (none) -> LCSC; now not fitted
- BZ1: value (none) -> Buzzer; footprint (none) -> User_Footprints:XDCR_CMT-7525-80-SMT-TR
- C1, C2: value (none) -> 1u; footprint (none) -> User_Footprints:C_0603_1608Metric
- C3, C4: value (none) -> 18p; footprint (none) -> User_Footprints:C_0603_1608Metric
- C5, C6: value (none) -> 4u7; footprint (none) -> User_Footprints:C_0603_1608Metric
- D1: value (none) -> LED; footprint (none) -> LED_SMD:LED_0603_1608Metric; Manufacturer (none) -> XINGLIGHT; Notes (none) -> 20mA; Package (none) -> 0603; Part Number (none) -> XL-1608SURC-06
- J1: value (none) -> TC2050-IDC-NL; footprint (none) -> User_Footprints:TAG-CONNECT_TC2050-IDC-NL; Notes (none) -> Integrated; now not fitted
- J2: value (none) -> USB-C_Port; footprint (none) -> User_Footprints:GCT_USB4110GFA; Manufacturer (none) -> G-Switch; Notes (none) -> 5A; Package (none) -> SMD
- J3: value (none) -> TP4057; footprint (none) -> User_Footprints:SOT-23-6; Manufacturer (none) -> YONGYUTAI; Notes (none) -> 0.3V-6.5V 600mA; Package (none) -> SOT-23-6L
- Q1, Q2, Q3, Q4: value (none) -> HL-2301V; footprint (none) -> User_Footprints:SOT-23
- R1, R2, R5, R6: value (none) -> 5K1; footprint (none) -> User_Footprints:R_0603_1608Metric
- R10, R11, R15, R16, R17, R18, R19, R3, R8, R9: value (none) -> 1K; footprint (none) -> User_Footprints:R_0603_1608Metric
- R12, R13, R14, R7: value (none) -> 100K; footprint (none) -> User_Footprints:R_0603_1608Metric; Manufacturer (none) -> FOJAN; Notes (none) -> 100mW 5%; Package (none) -> 0603; Part Number (none) -> FRC0603J104 TS; Price (none) -> .0007; Vendor (none) -> LCSC; Website (none) -> https://www.lcsc.com/product-detail/Chip-Resistor-Surface-M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
- R4: value (none) -> 1K6; footprint (none) -> User_Footprints:R_0603_1608Metric; Manufacturer (none) -> VO; Notes (none) -> 100mW 5%; Package (none) -> 0603; Part Number (none) -> SCR0603J1K6; Price (none) -> .0005; Vendor (none) -> LCSC; Website (none) -> https://www.lcsc.com/product-detail/Chip-Resistor-Surface-M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
- SW1, SW2, SW3: value (none) -> SW_Push; footprint (none) -> User_Footprints:Oval_Button
- U1: value (none) -> BC833M; footprint (none) -> User_Footprints:XCVR_BC833M; Notes (none) -> nRF52833; Package (none) -> SMD

Commit message: Created hardware revision 0.3, sent to fab.
Parts:
- removed BZ1: Buzzer, User_Footprints:XDCR_CMT-7525-80-SMT-TR, symbol Device:Buzzer
- removed Q1, Q2, Q3, Q4: HL-2301V, User_Footprints:SOT-23, symbol User_Symbols:HL-2301V
- removed R10, R11, R15, R16, R17, R18, R19, R9: 1K, User_Footprints:R_0603_1608Metric, symbol Device:R
- removed R12, R13, R14: 100K, User_Footprints:R_0603_1608Metric, symbol Device:R
- added BZ2: Buzzer, User_Footprints:XDCR_CMT-7525-80-SMT-TR, symbol Device:Buzzer
- added C10, C7, C8: 100n, Capacitor_SMD:C_0603_1608Metric, symbol Device:C
- added C9: 1u, User_Footprints:C_0603_1608Metric, symbol Device:C
- added Q5, Q6, Q7: HL-2302V, Package_TO_SOT_SMD:SOT-23, symbol User_Symbols:HL-2302V
- added R20, R22: 1K, User_Footprints:R_0603_1608Metric, symbol Device:R
- added R21: 100K, User_Footprints:R_0603_1608Metric, symbol Device:R
- added R24, R27, R46, R48, R49, R50, R58, R59, R60, R62: 21, User_Footprints:R_0603_1608Metric, symbol Device:R
- added R25: 100, User_Footprints:R_0603_1608Metric, symbol Device:R
- added R28, R29, R47, R51, R61: 43, User_Footprints:R_0603_1608Metric, symbol Device:R
- added U2: DW01A, Package_TO_SOT_SMD:SOT-23-6, symbol Battery_Management:DW01A
- added U3: IS31FL3729, Package_DFN_QFN:QFN-32-1EP_4x4mm_P0.4mm_EP2.9x2.9mm_ThermalVias, symbol User_Symbols:IS31FL3729
- AE1: now fitted; now left out of the parts list
- BT1: LCSC Part Number (none) -> C3029440; Part Number WAFER-PH2.0-2PWB -> WAFER-PH2.0-2PWB
- BT2: LCSC Part Number (none) -> C5290176
- C1, C2: LCSC Part Number (none) -> C1592
- C3, C4: LCSC Part Number (none) -> C5137620
- C5, C6: LCSC Part Number (none) -> C7503506; Part Number CSA0603X5R475K6R3JT -> CGA0603X5R475K6R3JT; Website https://www.lcsc.com/product-detail/Multilayer-Ceramic-Capacitors-MLCC-SMD-SMT_HRE-CSA0603X5R475K6R3JT_C3015159.html -> https://www.lcsc.com/product-detail/Multilayer-Ceramic-Capacitors-MLCC-SMD-SMT_HRE-CGA0603X5R475K6R3JT_C7503506.html?s_z=n_CSA0603X5R475K6R3JT
- D1: LCSC Part Number (none) -> C965799
- J1: Manufacturer (none) -> Tag-Connect; Package (none) -> N/a; Part Number (none) -> TC2050-IDC; Price (none) -> .00; Vendor (none) -> Tag-Connect; Website (none) -> https://www.tag-connect.com/product/tc2050-idc-tag-connect-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; now fitted
- J2: LCSC Part Number (none) -> C963371
- J3: LCSC Part Number (none) -> C20199358
- R1, R2: LCSC Part Number (none) -> C105580
- R3: LCSC Part Number (none) -> C2907113
- R4: value 1K6 -> 5K1; LCSC Part Number (none) -> C105580; Manufacturer VO -> YAGEO; Notes 100mW 5% -> 100mW 1%; Part Number SCR0603J1K6 -> RC0603FR-075K1L; Price .0005 -> .0013; Website https://www.lcsc.com/product-detail/Chip-Resistor-Surface-Mount_VO-SCR0603J1K6_C3017732.html -> https://www.lcsc.com/product-detail/Chip-Resistor-Surface-Mount_YAGEO-RC0603FR-075K1L_C105580.html
- R5, R6: value 5K1 -> 2K; LCSC Part Number (none) -> C2907137; Manufacturer YAGEO -> Fojan; Notes 100mW 1% -> 100mW 5%; Part Number RC0603FR-075K1L -> FRC0603J202 TS; Price .0013 -> .0008; Website https://www.lcsc.com/product-detail/Chip-Resistor-Surface-Mount_YAGEO-RC0603FR-075K1L_C105580.html -> https://www.lcsc.com/product-detail/Chip-Resistor-Surface-Mount_FOJAN-FRC0603J202-TS_C2907137.html
- R7: LCSC Part Number (none) -> C2907088
- R8: value 1K -> 10K; LCSC Part Number (none) -> C2930027; Notes 100mW 1% -> 100mW 5%; Part Number FRC0603J102 TS -> FRC0603J103 TS; Website https://www.lcsc.com/product-detail/Chip-Resistor-Surface-Mount_FOJAN-FRC0603J102-TS_C2907113.html -> https://www.lcsc.com/product-detail/Chip-Resistor-Surface-Mount_FOJAN-FRC0603J103-TS_C2930027.html
- SW1, SW2, SW3: footprint User_Footprints:Oval_Button -> User_Footprints:SW4_1437565_TEC; LCSC Part Number (none) -> C318888; Manufacturer BZCN -> XKB Connection; Part Number TSA016A2526A -> TS-1187A-C-D-B; Price .0136 -> .0368; Website https://www.lcsc.com/product-detail/Tactile-Switches_BZCN-T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 -> https://www.lcsc.com/product-detail/Tactile-Switches_XKB-Co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
Connections:
- net GND: now also R7.2, R8.2, C7.2, C8.2, C9.2, Q5.2 (S), Q6.2 (S), R21.2, R22.1, U3.24 (GND), U3.28 (AD), U3.33 (GND), U3.9 (GND); no longer BT1.2 (-), BT2.2 (-), J3.5 (STDBY), R4.2, R6.2
- net VBAT: now also U1.13 (VDDH), BZ2.1 (+), C7.1, C9.1, R25.1, U3.23 (VCC)
- net VBUS: no longer U1.13 (VDDH)
- net VDD: now also R5.1, R6.1; no longer R7.1
- net at R8.1: now also U3.25 (ISET); no longer U1.07 (P030)
- net at U1.03 (P002): now also R20.1
- net at U1.06 (P029): now also SW3.2
- net SDB: now reaches U1.10 (P005)
- net SDB: now also R7.1, C8.1, U3.29 (SDB)
- net SCL: now reaches U1.11 (P109)
- net SCL: now also R6.2, U3.27 (SCL)
- net SDA: now reaches U1.12 (P011)
- net SDA: now also R5.2, U3.26 (SDA)
- net at SW2.2: now also U1.07 (P030); no longer U1.17 (P018)
- net at SW1.2: now also U1.02 (P003); no longer U1.20 (P017)
- net at U1.21 (P020): no longer SW3.2
- new net: R61.1, U3.31 (CS2)
- new net: R51.1, U3.3 (CS6)
- new net: R22.2, U2.2 (CS)
- new net: BT1.2 (-), BT2.2 (-), C10.2, Q7.2 (S), U2.6 (GND)
- new net: R29.1, U3.10 (CS12)
- new net: Q7.1 (G), U2.1 (OD)
- new net: Q6.3 (D), Q7.3 (D)
- new net: C10.1, R25.2, U2.5 (VCC)
- new net: R59.1, U3.1 (CS4)
- new net: R27.1, U3.11 (CS13)
- new net: R24.1, U3.12 (CS14)
- new net: R28.1, U3.13 (CS15)
- new net: R58.1, U3.2 (CS5)
- new net: R62.1, U3.30 (CS1)
- new net: R60.1, U3.32 (CS3)
- new net: R50.1, U3.4 (CS7)
- new net: R49.1, U3.5 (CS8)
- new net: R48.1, U3.6 (CS9)
- new net: R47.1, U3.7 (CS10)
- new net: R46.1, U3.8 (CS11)
- new net: Q5.1 (G), R20.2, R21.1
- new net: J3.5 (STDBY), R4.2
- new net: Q6.1 (G), U2.3 (OC)
- new net: BZ2.2 (-), Q5.3 (D)
- new net BLUE_BOTTOM: R62.2
- new net BLUE_LEFT_1: R27.2
- new net BLUE_LEFT_2: R48.2
- new net BLUE_RIGHT_1: R50.2
- new net BLUE_RIGHT_2: R59.2
- new net GREEN_BOTTOM: R60.2
- new net GREEN_LEFT_1: R24.2
- new net GREEN_LEFT_2: R46.2
- new net GREEN_RIGHT_1: R49.2
- new net GREEN_RIGHT_2: R58.2
- new net RED_BOTTOM: R61.2
- new net RED_LEFT_1: R28.2
- new net RED_LEFT_2: R29.2
- new net RED_RIGHT_1: R47.2
- new net RED_RIGHT_2: R51.2
- new net Segment_A: U3.19 (SW4)
- new net Segment_B: U3.18 (SW5)
- new net Segment_C: U3.15 (SW8)
- new net Segment_D: U3.14 (SW9/CS16)
- new net Segment_E: U3.17 (SW6)
- new net Segment_F: U3.20 (SW3)
- new net Segment_G: U3.16 (SW7)
- new net Segment_H: U3.22 (SW1)
- new net Segment_I: U3.21 (SW2)
- no-connect marks 5 -> 11
Other:
- sheet Right_Display renamed Left_Segment_1
- removed sheet Bottom_Display
- removed sheet Left_Display
- added sheet Bottom_Segment (Bottom_Segment.kicad_sch)
- added sheet Left_Segment_2 (Left_Segment_2.kicad_sch)
- added sheet Right_Segment_1 (Right_Segment_1.kicad_sch)
- added sheet Right_Segment_2 (Right_Segment_2.kicad_sch)
- sheet Left_Segment_1: file Right_Display.kicad_sch -> Left_Segment_1.kicad_sch
- sheet Left_Segment_1 ports: added BLUE, GREEN, RED, Segment_A, Segment_B, Segment_C, Segment_D, Segment_E, Segment_F, Segment_G, Segment_H, Segment_I; removed R1_DIN, R2_DIN, R_VDD, R_VSS
- moved on the sheet: BT1, BT2, C1, C2, C3, C4, C5, C6, D1, J2, J3, R1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

Commit message: Fixed missing ground connection
Connections:
- net GND: now also J3.5 (STDBY), R4.2
Changed lines of the file:
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@@
 (kicad_sch
-	(version 20231120)
+	(version 20250114)
 	(generator "eeschema")
-	(generator_version "8.0")
+	(generator_version "9.0")
 	(paper "USLedger")
 	(junction
@@
 	)
 	(junction
+		(at 118.11 87.63)
+		(diameter 0)
+		(color 0 0 0 0)
+	)
+	(junction
 		(at 66.04 113.03)
 		(diameter 0)
@@
 	(wire
 		(pts
+			(xy 118.11 87.63) (xy 132.08 87.63)
+		)
+		(stroke
+			(width 0)
+			(type default)
+		)
+	)
+	(wire
+		(pts
 			(xy 86.36 85.09) (xy 86.36 87.63)
 		)
@@
 	(wire
 		(pts
-			(xy 104.14 87.63) (xy 132.08 87.63)
+			(xy 104.14 87.63) (xy 118.11 87.63)
 		)
 		(stroke
@@
 		(at 326.39 196.215)
 		(size 45.72 29.21)
+		(exclude_from_sim no)
+		(in_bom yes)
+		(on_board yes)
+		(dnp no)
 		(stroke
 			(width 0.1524)
@@
 		(at 60.96 195.58)
 		(size 45.72 29.21)
+		(exclude_from_sim no)
+		(in_bom yes)
+		(on_board yes)
+		(dnp no)
 		(stroke
 			(width 0.1524)
@@
 		(at 148.59 194.945)
 		(size 45.72 29.21)
+		(exclude_from_sim no)
+		(in_bom yes)
+		(on_board yes)
+		(dnp no)
 		(stroke
 			(width 0.1524)
@@
 		(at 210.82 234.95)
 		(size 45.72 29.21)
+		(exclude_from_sim no)
+		(in_bom yes)
+		(on_board yes)
+		(dnp no)
 		(stroke
 			(width 0.1524)
@@
 		(at 238.76 197.485)
 		(size 45.72 29.21)
+		(exclude_from_sim no)
+		(in_bom yes)
+		(on_board yes)
+		(dnp no)
 		(stroke
 			(width 0.1524)
@@
 		)
 	)
+	(embedded_fonts no)
 )
